File: asic/e-class-aardonyx/board/Board_Design/power.sch (KiCad schematic (older format))
At the start: 30 parts, among them J1 12V, SW1 SW_SPST, U7 TPS62086RLTR, U8 TPS54627DDAR, U9 TPS62061DSGR

Commit message: update
Parts:
- added C65: 47UF, symbol aardonyx:C_Small
- renumbered C45 to C63, C55 to C64, C47 to C66, C49 to C67, C59 to C68, C52 to C69, C60 to C70, C46 to C71, C48 to C72, C50 to C73, C51 to C74, C53 to C75, C54 to C76, C56 to C77, C57 to C78, C58 to C79, J1 to J8, L3 to L1, L1 to L2, L2 to L3, R15 to R70, R16 to R71, R11 to R72, R12 to R73, R13 to R74, R14 to R75, U7 to U10, U8 to U11
Connections:
- net GNDREF: now also C65.2
- net at C66.1, C67.1, SW1.2 (B): now also C65.1
Other:
- moved on the sheet: C66, C67
