File: asic/e-class-aardonyx/board/Board_Design/ftdi.sch (KiCad schematic (older format))
At the start: 28 parts, among them J2 Micro_USB, U3 FT2232H, Y1 12MHz

Commit message: update
Parts:
- gave numbers to parts that had none: 1
- renumbered C11 to C28, C12 to C29, C13 to C30, C14 to C31, C15 to C32, C16 to C33, C17 to C34, C18 to C35, C19 to C36, C20 to C37, C21 to C38, C22 to C39, C23 to C40, C24 to C41, C25 to C42, C26 to C43, R1 to R60, R2 to R61, R3 to R62, Y1 to Y2
Changed lines of the file:
@@
 	5450 2550 5350 2550
 $Comp
-L aardonyx:C_Small C20
+L aardonyx:C_Small C37
 U 1 1 5DB80465
 P 4850 2350
-F 0 "C20" H 4850 2450 50  0000 L CNN
+F 0 "C37" H 4850 2450 50  0000 L CNN
 F 1 "0.1uF" H 4850 2250 50  0000 L CNN
 F 2 "" H 4850 2350 50  0001 C CNN
@@
 $EndComp
 $Comp
-L aardonyx:C_Small C19
+L aardonyx:C_Small C36
 U 1 1 5DB818DD
 P 4550 2350
-F 0 "C19" H 4550 2450 50  0000 L CNN
+F 0 "C36" H 4550 2450 50  0000 L CNN
 F 1 "4.7uF" H 4550 2250 50  0000 L CNN
 F 2 "" H 4550 2350 50  0001 C CNN
@@
 $EndComp
 $Comp
-L aardonyx:C_Small C18
+L aardonyx:C_Small C35
 U 1 1 5DB8354B
 P 4250 1850
-F 0 "C18" H 4250 1950 50  0000 L CNN
+F 0 "C35" H 4250 1950 50  0000 L CNN
 F 1 "0.1uF" H 4250 1750 50  0000 L CNN
 F 2 "" H 4250 1850 50  0001 C CNN
@@
 $EndComp
 $Comp
-L aardonyx:C_Small C15
+L aardonyx:C_Small C32
 U 1 1 5DB83551
 P 3950 1850
-F 0 "C15" H 3950 1950 50  0000 L CNN
+F 0 "C32" H 3950 1950 50  0000 L CNN
 F 1 "4.7uF" H 3950 1750 50  0000 L CNN
 F 2 "" H 3950 1850 50  0001 C CNN
@@
 	6750 4850 7400 4850
 $Comp
-L aardonyx:C_Small C14
+L aardonyx:C_Small C31
 U 1 1 5DB9AA70
 P 3750 3400
-F 0 "C14" H 3750 3500 50  0000 L CNN
+F 0 "C31" H 3750 3500 50  0000 L CNN
 F 1 "0.1uF" H 3750 3300 50  0000 L CNN
 F 2 "" H 3750 3400 50  0001 C CNN
@@
 $EndComp
 $Comp
-L aardonyx:C_Small C12
+L aardonyx:C_Small C29
 U 1 1 5DB9AA76
 P 3450 3400
-F 0 "C12" H 3450 3500 50  0000 L CNN
+F 0 "C29" H 3450 3500 50  0000 L CNN
 F 1 "4.7uF" H 3450 3300 50  0000 L CNN
 F 2 "" H 3450 3400 50  0001 C CNN
@@
 $EndComp
 $Comp
-L aardonyx:C_Small C17
+L aardonyx:C_Small C34
 U 1 1 5DBA0960
 P 4050 3400
-F 0 "C17" H 4050 3500 50  0000 L CNN
+F 0 "C34" H 4050 3500 50  0000 L CNN
 F 1 "0.1uF" H 4050 3300 50  0000 L CNN
 F 2 "" H 4050 3400 50  0001 C CNN
@@
 Connection ~ 4250 7150
 $Comp
-L aardonyx:GND #PWR016
+L aardonyx:GND #PWR025
 U 1 1 5DDDD200
 P 4250 7350
-F 0 "#PWR016" H 4250 7100 50  0001 C CNN
+F 0 "#PWR025" H 4250 7100 50  0001 C CNN
 F 1 "GND" H 4255 7177 50  0000 C CNN
 F 2 "" H 4250 7350 50  0001 C CNN
@@
 $EndComp
 $Comp
-L aardonyx:GND #PWR013
+L aardonyx:GND #PWR022
 U 1 1 5DDDE1C1
 P 3450 3650
-F 0 "#PWR013" H 3450 3400 50  0001 C CNN
+F 0 "#PWR022" H 3450 3400 50  0001 C CNN
 F 1 "GND" H 3455 3477 50  0000 C CNN
 F 2 "" H 3450 3650 50  0001 C CNN
@@
 $EndComp
 $Comp
-L aardonyx:GND #PWR014
+L aardonyx:GND #PWR023
 U 1 1 5DDE30A8
 P 3950 2650
-F 0 "#PWR014" H 3950 2400 50  0001 C CNN
+F 0 "#PWR023" H 3950 2400 50  0001 C CNN
 F 1 "GND" H 3955 2477 50  0000 C CNN
 F 2 "" H 3950 2650 50  0001 C CNN
@@
 $EndComp
 $Comp
-L aardonyx:GND #PWR015
+L aardonyx:GND #PWR024
 U 1 1 5DDE529E
 P 4250 4950
-F 0 "#PWR015" H 4250 4700 50  0001 C CNN
+F 0 "#PWR024" H 4250 4700 50  0001 C CNN
 F 1 "GND" H 4255 4777 50  0000 C CNN
 F 2 "" H 4250 4950 50  0001 C CNN
@@
 $EndComp
 $Comp
-L aardonyx:V3P3 #PWR012
+L aardonyx:V3P3 #PWR021
 U 1 1 5DDE84A3
 P 3200 1350
-F 0 "#PWR012" H 3350 1300 50  0001 C CNN
+F 0 "#PWR021" H 3350 1300 50  0001 C CNN
 F 1 "V3P3" H 3205 1525 50  0000 C CNN
 F 2 "" H 3200 1350 50  0001 C CNN
@@
 $EndComp
 $Comp
-L aardonyx:VCORE_FTDI #PWR011
+L aardonyx:VCORE_FTDI #PWR020
 U 1 1 5E3E23EC
 P 2850 3100
-F 0 "#PWR011" H 3000 3050 50  0001 C CNN
+F 0 "#PWR020" H 3000 3050 50  0001 C CNN
 F 1 "VCORE_FTDI" H 2855 3275 50  0000 C CNN
 F 2 "" H 2850 3100 50  0001 C CNN
@@
 	6050 2350 6050 2550
 $Comp
-L aardonyx:V3P3 #PWR018
+L aardonyx:V3P3 #PWR027
 U 1 1 5DDE7896
 P 6050 2350
-F 0 "#PWR018" H 6200 2300 50  0001 C CNN
+F 0 "#PWR027" H 6200 2300 50  0001 C CNN
 F 1 "V3P3" H 6055 2525 50  0000 C CNN
 F 2 "" H 6050 2350 50  0001 C CNN
@@
 $EndComp
 $Comp
-L aardonyx:VCORE_FTDI #PWR017
+L aardonyx:VCORE_FTDI #PWR026
 U 1 1 5E3E1553
 P 5550 2350
-F 0 "#PWR017" H 5700 2300 50  0001 C CNN
+F 0 "#PWR026" H 5700 2300 50  0001 C CNN
 F 1 "VCORE_FTDI" H 5555 2525 50  0000 C CNN
 F 2 "" H 5550 2350 50  0001 C CNN
@@
 $EndComp
 $Comp
-L aardonyx:C_Small C21
+L aardonyx:C_Small C38
 U 1 1 5E439A51
 P 8000 1650
-F 0 "C21" H 8000 1750 50  0000 L CNN
+F 0 "C38" H 8000 1750 50  0000 L CNN
 F 1 "0.1uF" H 8000 1550 50  0000 L CNN
 F 2 "" H 8000 1650 50  0001 C CNN
@@
 $EndComp
 $Comp
-L aardonyx:C_Small C22
+L aardonyx:C_Small C39
 U 1 1 5E43C0DA
 P 8250 1650
-F 0 "C22" H 8250 1750 50  0000 L CNN
+F 0 "C39" H 8250 1750 50  0000 L CNN
 F 1 "0.1uF" H 8250 1550 50  0000 L CNN
 F 2 "" H 8250 1650 50  0001 C CNN
@@
 $EndComp
 $Comp
-L aardonyx:C_Small C23
+L aardonyx:C_Small C40
 U 1 1 5E43E6EE
 P 8500 1650
-F 0 "C23" H 8500 1750 50  0000 L CNN
+F 0 "C40" H 8500 1750 50  0000 L CNN
 F 1 "0.1uF" H 8500 1550 50  0000 L CNN
 F 2 "" H 8500 1650 50  0001 C CNN
@@
 	8250 1850 8500 1850
 $Comp
-L aardonyx:VCORE_FTDI #PWR019
+L aardonyx:VCORE_FTDI #PWR030
 U 1 1 5E454E04
 P 8000 1350
-F 0 "#PWR019" H 8150 1300 50  0001 C CNN
+F 0 "#PWR030" H 8150 1300 50  0001 C CNN
 F 1 "VCORE_FTDI" H 8005 1525 50  0000 C CNN
 F 2 "" H 8000 1350 50  0001 C CNN
@@
 $EndComp
 $Comp
-L aardonyx:GND #PWR020
+L aardonyx:GND #PWR031
 U 1 1 5E456D74
 P 8500 1950
-F 0 "#PWR020" H 8500 1700 50  0001 C CNN
+F 0 "#PWR031" H 8500 1700 50  0001 C CNN
 F 1 "GND" H 8505 1777 50  0000 C CNN
 F 2 "" H 8500 1950 50  0001 C CNN
@@
 	9650 1950 9650 1850
 $Comp
-L aardonyx:GND #PWR024
+L aardonyx:GND #PWR033
 U 1 1 5E456003
 P 9650 1950
-F 0 "#PWR024" H 9650 1700 50  0001 C CNN
+F 0 "#PWR033" H 9650 1700 50  0001 C CNN
 F 1 "GND" H 9655 1777 50  0000 C CNN
 F 2 "" H 9650 1950 50  0001 C CNN
@@
 $EndComp
 $Comp
-L aardonyx:V3P3 #PWR022
+L aardonyx:V3P3 #PWR032
 U 1 1 5E4559CC
 P 8900 1350
-F 0 "#PWR022" H 9050 1300 50  0001 C CNN
+F 0 "#PWR032" H 9050 1300 50  0001 C CNN
 F 1 "V3P3" H 8905 1525 50  0000 C CNN
 F 2 "" H 8900 1350 50  0001 C CNN
@@
 	8900 1550 8900 1450
 $Comp
-L aardonyx:C_Small C26
+L aardonyx:C_Small C43
 U 1 1 5E437345
 P 9400 1650
-F 0 "C26" H 9400 1750 50  0000 L CNN
+F 0 "C43" H 9400 1750 50  0000 L CNN
 F 1 "0.1uF" H 9400 1550 50  0000 L CNN
 F 2 "" H 9400 1650 50  0001 C CNN
@@
 $EndComp
 $Comp
-L aardonyx:C_Small C25
+L aardonyx:C_Small C42
 U 1 1 5E434CF2
 P 9150 1650
-F 0 "C25" H 9150 1750 50  0000 L CNN
+F 0 "C42" H 9150 1750 50  0000 L CNN
 F 1 "0.1uF" H 9150 1550 50  0000 L CNN
 F 2 "" H 9150 1650 50  0001 C CNN
@@
 $EndComp
 $Comp
-L aardonyx:C_Small C24
+L aardonyx:C_Small C41
 U 1 1 5E432586
 P 8900 1650
-F 0 "C24" H 8900 1750 50  0000 L CNN
+F 0 "C41" H 8900 1750 50  0000 L CNN
 F 1 "0.1uF" H 8900 1550 50  0000 L CNN
 F 2 "" H 8900 1650 50  0001 C CNN
@@
 $EndComp
 $Comp
-L aardonyx:R_US R1
+L aardonyx:R_US R60
 U 1 1 5E4FC879
 P 4250 4700
-F 0 "R1" H 4300 4800 50  0000 L CNN
+F 0 "R60" H 4300 4800 50  0000 L CNN
 F 1 "12K" H 4250 4550 50  0000 L CNN
 F 2 "" V 4290 4690 50  0001 C CNN
@@
 	1050 4450 1050 4350
 $Comp
-L aardonyx:GND #PWR08
+L aardonyx:GND #PWR017
 U 1 1 5E51637D
 P 1050 4650
-F 0 "#PWR08" H 1050 4400 50  0001 C CNN
+F 0 "#PWR017" H 1050 4400 50  0001 C CNN
 F 1 "GND" H 1055 4477 50  0000 C CNN
 F 2 "" H 1050 4650 50  0001 C CNN
@@
 	1350 3750 1450 3750
 $Comp
-L aardonyx:C_Small C11
+L aardonyx:C_Small C28
 U 1 1 5E522768
 P 1650 3500
-F 0 "C11" H 1650 3600 50  0000 L CNN
+F 0 "C28" H 1650 3600 50  0000 L CNN
 F 1 "4.7uF" H 1650 3400 50  0000 L CNN
 F 2 "" H 1650 3500 50  0001 C CNN
@@
 $EndComp
 $Comp
-L aardonyx:GND #PWR010
+L aardonyx:GND #PWR019
 U 1 1 5E5269D8
 P 1650 3650
-F 0 "#PWR010" H 1650 3400 50  0001 C CNN
+F 0 "#PWR019" H 1650 3400 50  0001 C CNN
 F 1 "GND" H 1655 3477 50  0000 C CNN
 F 2 "" H 1650 3650 50  0001 C CNN
@@
 Connection ~ 1450 3350
 $Comp
-L aardonyx:VBUS #PWR09
+L aardonyx:VBUS #PWR018
 U 1 1 5E53F521
 P 1450 3000
-F 0 "#PWR09" H 1600 2950 50  0001 C CNN
+F 0 "#PWR018" H 1600 2950 50  0001 C CNN
 F 1 "VBUS" H 1455 3175 50  0000 C CNN
 F 2 "" H 1450 3000 50  0001 C CNN
@@
 	2200 3950 4350 3950
 $Comp
-L aardonyx:Crystal Y1
+L aardonyx:Crystal Y2
 U 1 1 5E59521C
 P 3700 6450
-F 0 "Y1" H 3700 6718 50  0000 C CNN
+F 0 "Y2" H 3700 6718 50  0000 C CNN
 F 1 "12MHz" H 3700 6627 50  0000 C CNN
 F 2 "" H 3700 6450 50  0001 C CNN
@@
 $EndComp
 $Comp
-L aardonyx:C_Small C16
+L aardonyx:C_Small C33
 U 1 1 5E5A19BF
 P 3950 6750
-F 0 "C16" H 3950 6850 50  0000 L CNN
+F 0 "C33" H 3950 6850 50  0000 L CNN
 F 1 "30pF" H 3950 6650 50  0000 L CNN
 F 2 "" H 3950 6750 50  0001 C CNN
@@
 $EndComp
 $Comp
-L aardonyx:C_Small C13
+L aardonyx:C_Small C30
 U 1 1 5E5A728B
 P 3450 6750
-F 0 "C13" H 3450 6850 50  0000 L CNN
+F 0 "C30" H 3450 6850 50  0000 L CNN
 F 1 "30pF" H 3450 6650 50  0000 L CNN
 F 2 "" H 3450 6750 50  0001 C CNN
@@
 	3450 6050 4350 6050
 $Comp
-L aardonyx:R_US R2
+L aardonyx:R_US R61
 U 1 1 5E5E8E68
 P 7100 3700
-F 0 "R2" H 7168 3746 50  0000 L CNN
+F 0 "R61" H 7168 3746 50  0000 L CNN
 F 1 "1K" H 7168 3655 50  0000 L CNN
 F 2 "" V 7140 3690 50  0001 C CNN
@@
 $EndComp
 $Comp
-L aardonyx:R_US R3
+L aardonyx:R_US R62
 U 1 1 5E5EA6FB
 P 7200 2650
-F 0 "R3" H 7268 2696 50  0000 L CNN
+F 0 "R62" H 7268 2696 50  0000 L CNN
 F 1 "1K" H 7268 2605 50  0000 L CNN
 F 2 "" V 7240 2640 50  0001 C CNN
@@
 	7200 3250 7550 3250
 $Comp
-L aardonyx:V3P3 #PWR023
+L aardonyx:V3P3 #PWR029
 U 1 1 5E61CC4F
 P 7200 2400
-F 0 "#PWR023" H 7350 2350 50  0001 C CNN
+F 0 "#PWR029" H 7350 2350 50  0001 C CNN
 F 1 "V3P3" H 7205 2575 50  0000 C CNN
 F 2 "" H 7200 2400 50  0001 C CNN
@@
 	7200 2400 7200 2500
 $Comp
-L aardonyx:GND #PWR021
+L aardonyx:GND #PWR028
 U 1 1 5E6299DC
 P 7100 3950
-F 0 "#PWR021" H 7100 3700 50  0001 C CNN
+F 0 "#PWR028" H 7100 3700 50  0001 C CNN
 F 1 "GND" H 7105 3777 50  0000 C CNN
 F 2 "" H 7100 3950 50  0001 C CNN
@@
 	9650 1850 9650 1750
 $Comp
-L aardonyx:C_Small C?
+L aardonyx:C_Small C44
 U 1 1 5DD4FE8E
 P 9650 1650
-F 0 "C?" H 9650 1750 50  0000 L CNN
+F 0 "C44" H 9650 1750 50  0000 L CNN
 F 1 "0.1uF" H 9650 1550 50  0000 L CNN
 F 2 "" H 9650 1650 50  0001 C CNN

Commit message: update
Parts:
- added R60: 12K, symbol aardonyx:R_US
- added R63, R64, R66, R67, R68, R69, R70, R71, R72, R73, R74, R75, R76, R77: 1K, symbol aardonyx:R_US
- renumbered R60 to R61, R61 to R65
Connections:
- net labels added: FT_RESET
- wire segments 152 -> 205
Other:
- moved on the sheet: C28, C29, C30, C31, C32, C33, C34, C35, C36, C37, D1, D2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

Commit message: update
Parts:
- renumbered C28 to C1, C37 to C10, C38 to C11, C39 to C12, C40 to C13, C41 to C14, C42 to C15, C43 to C16, C44 to C17, C29 to C2, C30 to C3, C31 to C4, C32 to C5, C33 to C6, C34 to C7, C35 to C8, C36 to C9, J2 to J1, R60 to R1, R69 to R10, R70 to R11, R71 to R12, R72 to R13, R73 to R14, R74 to R15, R75 to R16, R76 to R17, R77 to R18, R61 to R2, R62 to R3, R63 to R4, R64 to R5, R65 to R6, R66 to R7, R67 to R8, R68 to R9, U3 to U1, Y2 to Y1
Connections:
- wire segments 205 -> 204
- no-connect marks 0 -> 27
Other:
- moved on the sheet: R3, R4

Commit message: update
Parts:
- R10, R11, R12, R13, R14, R16, R18, R5, R6, R7, R8, R9: Field4 (none) -> NA
Changed lines of the file:
@@
 F 2 "" V 9390 3890 50  0001 C CNN
 F 3 "~" H 9350 3900 50  0001 C CNN
+F 4 "NA" H 9450 3750 50  0000 C CNN "Field4"
 	1    9350 3900
 	1    0    0    -1
@@
 F 2 "" V 9390 2990 50  0001 C CNN
 F 3 "~" H 9350 3000 50  0001 C CNN
+F 4 "NA" H 9450 2850 50  0000 C CNN "Field4"
 	1    9350 3000
 	1    0    0    -1
@@
 F 2 "" V 9640 3890 50  0001 C CNN
 F 3 "~" H 9600 3900 50  0001 C CNN
+F 4 "NA" H 9650 3750 50  0000 C CNN "Field4"
 	1    9600 3900
 	1    0    0    -1
@@
 F 2 "" V 9640 2990 50  0001 C CNN
 F 3 "~" H 9600 3000 50  0001 C CNN
+F 4 "NA" H 9650 2850 50  0000 C CNN "Field4"
 	1    9600 3000
 	1    0    0    -1
@@
 F 2 "" V 9890 3890 50  0001 C CNN
 F 3 "~" H 9850 3900 50  0001 C CNN
+F 4 "NA" H 9900 3750 50  0000 C CNN "Field4"
 	1    9850 3900
 	1    0    0    -1
@@
 F 2 "" V 9890 2990 50  0001 C CNN
 F 3 "~" H 9850 3000 50  0001 C CNN
+F 4 "NA" H 9900 2850 50  0000 C CNN "Field4"
 	1    9850 3000
 	1    0    0    -1
@@
 F 2 "" V 10140 3890 50  0001 C CNN
 F 3 "~" H 10100 3900 50  0001 C CNN
+F 4 "NA" H 10150 3750 50  0000 C CNN "Field4"
 	1    10100 3900
 	1    0    0    -1
@@
 F 2 "" V 10390 3890 50  0001 C CNN
 F 3 "~" H 10350 3900 50  0001 C CNN
+F 4 "NA" H 10400 3750 50  0000 C CNN "Field4"
 	1    10350 3900
 	1    0    0    -1
@@
 F 2 "" V 9840 5840 50  0001 C CNN
 F 3 "~" H 9800 5850 50  0001 C CNN
+F 4 "NA" H 9900 5700 50  0000 C CNN "Field4"
 	1    9800 5850
 	1    0    0    -1
@@
 F 2 "" V 9840 4940 50  0001 C CNN
 F 3 "~" H 9800 4950 50  0001 C CNN
+F 4 "NA" H 9900 4800 50  0000 C CNN "Field4"
 	1    9800 4950
 	1    0    0    -1
@@
 F 2 "" V 10090 5840 50  0001 C CNN
 F 3 "~" H 10050 5850 50  0001 C CNN
+F 4 "NA" H 10150 5700 50  0000 C CNN "Field4"
 	1    10050 5850
 	1    0    0    -1
@@
 F 2 "" V 10090 4940 50  0001 C CNN
 F 3 "~" H 10050 4950 50  0001 C CNN
+F 4 "NA" H 10150 4800 50  0000 C CNN "Field4"
 	1    10050 4950
 	1    0    0    -1

Commit message: update
Parts:
- added J2: Conn_1x8, symbol aardonyx:Conn_1x8
- added J3: Conn_1x3_M, symbol aardonyx:Conn_1x3_M
Connections:
- net GNDREF: now also J2.8 (Pin_8), J3.3 (Pin_3)
- net TCK: now also J2.2 (Pin_2)
- net TDI: now also J2.3 (Pin_3)
- net TDO: now also J2.4 (Pin_4)
- net TMS: now also J2.5 (Pin_5)
- net TRST: now also J2.6 (Pin_6)
- net UART0_RX: now also J3.1 (Pin_1)
- net UART0_TX: now also J3.2 (Pin_2)
- no-connect marks 27 -> 28
Changed lines of the file:
@@
 encoding utf-8
 Sheet 2 7
-Title ""
+Title "AARDONYX_DEVELOPMENT_BOARD"
 Date ""
-Rev ""
-Comp ""
+Rev "R1V0"
+Comp "IIT_MADRAS"
 Comment1 ""
 Comment2 ""
@@
 	9650 1950 9650 1850
 $Comp
-L aardonyx:GND #PWR016
+L aardonyx:GND #PWR019
 U 1 1 5E456003
 P 9650 1950
-F 0 "#PWR016" H 9650 1700 50  0001 C CNN
+F 0 "#PWR019" H 9650 1700 50  0001 C CNN
 F 1 "GND" H 9655 1777 50  0000 C CNN
 F 2 "" H 9650 1950 50  0001 C CNN
@@
 $EndComp
 $Comp
-L aardonyx:V3P3 #PWR017
+L aardonyx:V3P3 #PWR020
 U 1 1 5E8AF826
 P 9850 2750
-F 0 "#PWR017" H 10000 2700 50  0001 C CNN
+F 0 "#PWR020" H 10000 2700 50  0001 C CNN
 F 1 "V3P3" H 9855 2925 50  0000 C CNN
 F 2 "" H 9850 2750 50  0001 C CNN
@@
 	9850 2750 9850 2800
 $Comp
-L aardonyx:GND #PWR018
+L aardonyx:GND #PWR021
 U 1 1 5E8AF82D
 P 9850 4150
-F 0 "#PWR018" H 9850 3900 50  0001 C CNN
+F 0 "#PWR021" H 9850 3900 50  0001 C CNN
 F 1 "GND" H 9855 3977 50  0000 C CNN
 F 2 "" H 9850 4150 50  0001 C CNN
@@
 	9800 5500 10050 5500
 $Comp
-L aardonyx:V3P3 #PWR019
+L aardonyx:V3P3 #PWR022
 U 1 1 5EAF36CD
 P 10050 4700
-F 0 "#PWR019" H 10200 4650 50  0001 C CNN
+F 0 "#PWR022" H 10200 4650 50  0001 C CNN
 F 1 "V3P3" H 10055 4875 50  0000 C CNN
 F 2 "" H 10050 4700 50  0001 C CNN
@@
 Connection ~ 10050 4750
 $Comp
-L aardonyx:GND #PWR020
+L aardonyx:GND #PWR023
 U 1 1 5EB089F3
 P 10050 6100
-F 0 "#PWR020" H 10050 5850 50  0001 C CNN
+F 0 "#PWR023" H 10050 5850 50  0001 C CNN
 F 1 "GND" H 10055 5927 50  0000 C CNN
 F 2 "" H 10050 6100 50  0001 C CNN
@@
 NoConn ~ 6850 6250
 NoConn ~ 6850 6350
+$Comp
+L aardonyx:Conn_1x8 J?
+U 1 1 5E5A2193
+P 8700 3450
+AR Path="/5D8B37DE/5E5A2193" Ref="J?"  Part="1"
+AR Path="/5D8B3761/5E5A2193" Ref="J2"  Part="1"
+F 0 "J2" H 8650 3850 50  0000 L CNN
+F 1 "Conn_1x8" H 8550 2950 50  0000 L CNN
+F 2 "" H 8700 3450 50  0001 C CNN
+F 3 "~" H 8700 3450 50  0001 C CNN
+	1    8700 3450
+	-1   0    0    -1
+$EndComp
+NoConn ~ 8900 3750
+$Comp
+L aardonyx:V3P3 #PWR016
+U 1 1 5E5B7921
+P 8950 2950
+F 0 "#PWR016" H 9100 2900 50  0001 C CNN
+F 1 "V3P3" H 8955 3125 50  0000 C CNN
+F 2 "" H 8950 2950 50  0001 C CNN
+F 3 "" H 8950 2950 50  0001 C CNN
+	1    8950 2950
+	1    0    0    -1
+$EndComp
+$Comp
+L aardonyx:GND #PWR017
+U 1 1 5E5C2614
+P 8950 4000
+F 0 "#PWR017" H 8950 3750 50  0001 C CNN
+F 1 "GND" H 8955 3827 50  0000 C CNN
+F 2 "" H 8950 4000 50  0001 C CNN
+F 3 "" H 8950 4000 50  0001 C CNN
+	1    8950 4000
+	1    0    0    -1
+$EndComp
+Wire Wire Line
+	8900 3850 8950 3850
+Wire Wire Line
+	8950 3850 8950 4000
+Wire Wire Line
+	8950 3150 8900 3150
+Wire Wire Line
+	8950 2950 8950 3150
+$Comp
+L aardonyx:GND #PWR018
+U 1 1 5E5FC240
+P 9200 5700
+F 0 "#PWR018" H 9200 5450 50  0001 C CNN
+F 1 "GND" H 9205 5527 50  0000 C CNN
+F 2 "" H 9200 5700 50  0001 C CNN
+F 3 "" H 9200 5700 50  0001 C CNN
+	1    9200 5700
+	1    0    0    -1
+$EndComp
+$Comp
+L aardonyx:Conn_1x3_M J?
+U 1 1 5E613B93
+P 8950 5500
+AR Path="/5D8B37DE/5E613B93" Ref="J?"  Part="1"
+AR Path="/5D8B3761/5E613B93" Ref="J3"  Part="1"
+F 0 "J3" H 8950 5700 50  0000 L CNN
+F 1 "Conn_1x3_M" H 8850 5300 50  0000 L CNN
+F 2 "" H 8950 5500 50  0001 C CNN
+F 3 "~" H 8950 5500 50  0001 C CNN
+	1    8950 5500
+	-1   0    0    -1
+$EndComp
+Wire Wire Line
+	9150 5600 9200 5600
+Wire Wire Line
+	9200 5600 9200 5700
 $EndSCHEMATC

Commit message: updare
Parts:
- added TP1, TP2: TestPoint, symbol aardonyx:TestPoint
- C3, C6: value 30pF -> 18PF
- R1: value 12K -> 1k
- R3, R4: value 1K -> 0E
- Y1: Field4 (none) -> 9B-12.000MAAJ-B
Connections:
- net at U1.36 (~SUSPEND): now also TP2.1
- net at U1.60 (~PWREN): now also TP1.1
- no-connect marks 28 -> 26
Changed lines of the file:
@@
 P 3800 6150
 F 0 "Y1" H 3800 6418 50  0000 C CNN
-F 1 "12MHz" H 3800 6327 50  0000 C CNN
+F 1 "12MHz" H 3800 6000 50  0000 C CNN
 F 2 "" H 3800 6150 50  0001 C CNN
-F 3 "~" H 3800 6150 50  0001 C CNN
+F 3 "" H 3800 6150 50  0001 C CNN
+F 4 "9B-12.000MAAJ-B " H 3950 6300 50  0000 C CNN "Field4"
 	1    3800 6150
 	1    0    0    -1
@@
 P 4050 6450
 F 0 "C6" H 4050 6550 50  0000 L CNN
-F 1 "30pF" H 4050 6350 50  0000 L CNN
+F 1 "18PF" H 4050 6350 50  0000 L CNN
 F 2 "" H 4050 6450 50  0001 C CNN
 F 3 "~" H 4050 6450 50  0001 C CNN
@@
 P 3550 6450
 F 0 "C3" H 3550 6550 50  0000 L CNN
-F 1 "30pF" H 3550 6350 50  0000 L CNN
+F 1 "18PF" H 3550 6350 50  0000 L CNN
 F 2 "" H 3550 6450 50  0001 C CNN
 F 3 "~" H 3550 6450 50  0001 C CNN
@@
 P 3800 4200
 F 0 "R1" H 3850 4300 50  0000 L CNN
-F 1 "12K" H 3800 4050 50  0000 L CNN
+F 1 "1k" H 3800 4050 50  0000 L CNN
 F 2 "" V 3840 4190 50  0001 C CNN
 F 3 "~" H 3800 4200 50  0001 C CNN
@@
 P 7150 4450
 F 0 "R3" V 7200 4550 50  0000 L CNN
-F 1 "1K" V 7200 4250 50  0000 L CNN
+F 1 "0E" V 7200 4250 50  0000 L CNN
 F 2 "" V 7190 4440 50  0001 C CNN
 F 3 "~" H 7150 4450 50  0001 C CNN
@@
 P 7150 4550
 F 0 "R4" V 7200 4650 50  0000 L CNN
-F 1 "1K" V 7200 4350 50  0000 L CNN
+F 1 "0E" V 7200 4350 50  0000 L CNN
 F 2 "" V 7190 4540 50  0001 C CNN
 F 3 "~" H 7150 4550 50  0001 C CNN
@@
 Text HLabel 7800 4450 2    50   Output ~ 0
 UART0_RX
-Text HLabel 7800 4550 2    50   Output ~ 0
+Text HLabel 7800 4550 2    50   Input ~ 0
 UART0_TX
 Wire Wire Line
@@
 NoConn ~ 6850 5950
 NoConn ~ 6850 6050
-NoConn ~ 6850 6250
-NoConn ~ 6850 6350
 $Comp
 L aardonyx:Conn_1x8 J?
@@
 Wire Wire Line
 	9200 5600 9200 5700
+$Comp
+L aardonyx:TestPoint TP1
+U 1 1 5E8C6648
+P 6900 6250
+F 0 "TP1" V 6900 6438 50  0000 L CNN
+F 1 "TestPoint" V 6945 6438 50  0001 L CNN
+F 2 "" H 7100 6250 50  0001 C CNN
+F 3 "~" H 7100 6250 50  0001 C CNN
+	1    6900 6250
+	0    1    1    0
+$EndComp
+$Comp
+L aardonyx:TestPoint TP2
+U 1 1 5E8D220A
+P 6900 6350
+F 0 "TP2" V 6900 6538 50  0000 L CNN
+F 1 "TestPoint" V 6945 6538 50  0001 L CNN
+F 2 "" H 7100 6350 50  0001 C CNN
+F 3 "~" H 7100 6350 50  0001 C CNN
+	1    6900 6350
+	0    1    1    0
+$EndComp
+Wire Wire Line
+	6850 6250 6900 6250
+Wire Wire Line
+	6900 6350 6850 6350
 $EndSCHEMATC
