File: asic/e-class-aardonyx/board/Board_Design/ftdi.sch (KiCad schematic (older format))
At the start: 47 parts, among them J1 Micro_USB, J2 Conn_1x8, J3 Conn_1x3_M, U1 FT2232H, Y1 12MHz

Commit message: update bom
Parts:
- FB1, FB2, FB3: Description (none) -> FERRITE BEAD 600 OHM 0603 1LN; Digikey PartNumber (none) -> 732-1593-1-ND; Manufactured Part Number (none) -> 742792651; Maufaturer (none) -> Würth Elektronik
- R3, R4: Description (none) -> RES SMD 0 OHM JUMPER 1/8W 0805; Digikey PartNumber (none) -> 541-0.0ACT-ND; Manufactured Part Number (none) -> CRCW08050000Z0EA; Maufaturer (none) -> Vishay Dale
- U1: Description (none) -> Single chip USB to UART (RS232, RS422 or RS485)
- Y1: Description (none) -> CRYSTAL 12.0000MHZ 20PF SMD; Digikey PartNumber (none) -> XC1298CT-ND; Manufactured Part Number (none) -> ECS-120-20-5PXDN-TR; Maufaturer (none) -> ECS Inc.
Changed lines of the file:
@@
 F 2 "" H 5650 4550 50  0001 C CNN
 F 3 "http://www.ftdichip.com/Products/ICs/FT2232H.html" H 5650 4550 50  0001 C CNN
+F 4 "Single chip USB to UART (RS232, RS422 or RS485)" H 5650 4550 50  0001 C CNN "Description"
 	1    5650 4550
 	1    0    0    -1
@@
 F 1 "600R" V 3504 1800 50  0000 C CNN
 F 2 "" V 3580 1800 50  0001 C CNN
-F 3 "~" H 3650 1800 50  0001 C CNN
+F 3 "https://www.digikey.in/product-detail/en/w%C3%BCrth-elektronik/742792651/732-1593-1-ND/1639537" H 3650 1800 50  0001 C CNN
+F 4 "FERRITE BEAD 600 OHM 0603 1LN" H 3650 1800 50  0001 C CNN "Description"
+F 5 "732-1593-1-ND" H 3650 1800 50  0001 C CNN "Digikey PartNumber"
+F 6 "742792651" H 3650 1800 50  0001 C CNN "Manufactured Part Number"
+F 7 "Würth Elektronik" H 3650 1800 50  0001 C CNN "Maufaturer"
 	1    3650 1800
 	0    1    1    0
@@
 F 1 "600R" V 3504 1350 50  0000 C CNN
 F 2 "" V 3580 1350 50  0001 C CNN
-F 3 "~" H 3650 1350 50  0001 C CNN
+F 3 "https://www.digikey.in/product-detail/en/w%C3%BCrth-elektronik/742792651/732-1593-1-ND/1639537" H 3650 1350 50  0001 C CNN
+F 4 "FERRITE BEAD 600 OHM 0603 1LN" H 3650 1350 50  0001 C CNN "Description"
+F 5 "732-1593-1-ND" H 3650 1350 50  0001 C CNN "Digikey PartNumber"
+F 6 "742792651" H 3650 1350 50  0001 C CNN "Manufactured Part Number"
+F 7 "Würth Elektronik" H 3650 1350 50  0001 C CNN "Maufaturer"
 	1    3650 1350
 	0    1    1    0
@@
 F 1 "600R" H 1350 2900 50  0000 C CNN
 F 2 "" V 1480 2900 50  0001 C CNN
-F 3 "~" H 1550 2900 50  0001 C CNN
+F 3 "https://www.digikey.in/product-detail/en/w%C3%BCrth-elektronik/742792651/732-1593-1-ND/1639537" H 1550 2900 50  0001 C CNN
+F 4 "FERRITE BEAD 600 OHM 0603 1LN" H 1550 2900 50  0001 C CNN "Description"
+F 5 "732-1593-1-ND" H 1550 2900 50  0001 C CNN "Digikey PartNumber"
+F 6 "742792651" H 1550 2900 50  0001 C CNN "Manufactured Part Number"
+F 7 "Würth Elektronik" H 1550 2900 50  0001 C CNN "Maufaturer"
 	1    1550 2900
 	-1   0    0    1
@@
 F 1 "12MHz" H 3800 6000 50  0000 C CNN
 F 2 "" H 3800 6150 50  0001 C CNN
-F 3 "" H 3800 6150 50  0001 C CNN
+F 3 "https://www.digikey.in/product-detail/en/ecs-inc/ECS-120-20-5PXDN-TR/XC1298CT-ND/827762" H 3800 6150 50  0001 C CNN
 F 4 "9B-12.000MAAJ-B " H 3950 6300 50  0000 C CNN "Field4"
+F 5 "CRYSTAL 12.0000MHZ 20PF SMD" H 3800 6150 50  0001 C CNN "Description"
+F 6 "XC1298CT-ND" H 3800 6150 50  0001 C CNN "Digikey PartNumber"
+F 7 "ECS-120-20-5PXDN-TR" H 3800 6150 50  0001 C CNN "Manufactured Part Number"
+F 8 "ECS Inc." H 3800 6150 50  0001 C CNN "Maufaturer"
 	1    3800 6150
 	1    0    0    -1
@@
 F 1 "0E" V 7200 4250 50  0000 L CNN
 F 2 "" V 7190 4440 50  0001 C CNN
-F 3 "~" H 7150 4450 50  0001 C CNN
+F 3 "https://www.digikey.com/product-detail/en/vishay-dale/CRCW08050000Z0EA/541-0-0ACT-ND/1180267" H 7150 4450 50  0001 C CNN
+F 4 " RES SMD 0 OHM JUMPER 1/8W 0805 " H 7150 4450 50  0001 C CNN "Description"
+F 5 " 541-0.0ACT-ND " H 7150 4450 50  0001 C CNN "Digikey PartNumber"
+F 6 " CRCW08050000Z0EA " H 7150 4450 50  0001 C CNN "Manufactured Part Number"
+F 7 "Vishay Dale" H 7150 4450 50  0001 C CNN "Maufaturer"
 	1    7150 4450
 	0    -1   -1   0
@@
 F 1 "0E" V 7200 4350 50  0000 L CNN
 F 2 "" V 7190 4540 50  0001 C CNN
-F 3 "~" H 7150 4550 50  0001 C CNN
+F 3 "https://www.digikey.com/product-detail/en/vishay-dale/CRCW08050000Z0EA/541-0-0ACT-ND/1180267" H 7150 4550 50  0001 C CNN
+F 4 " RES SMD 0 OHM JUMPER 1/8W 0805 " H 7150 4550 50  0001 C CNN "Description"
+F 5 " 541-0.0ACT-ND " H 7150 4550 50  0001 C CNN "Digikey PartNumber"
+F 6 " CRCW08050000Z0EA " H 7150 4550 50  0001 C CNN "Manufactured Part Number"
+F 7 "Vishay Dale" H 7150 4550 50  0001 C CNN "Maufaturer"
 	1    7150 4550
 	0    -1   -1   0

Commit message: update BOM
Parts:
- C1, C2, C5, C9: Description CAP TANT 4.7UF 10% 16V 1206 -> CAP CER 4.7UF 25V X7R 1206; Digikey PartNumber 399-3697-1-ND -> 399-8203-1-ND; Manufactured Part Number T491A475K016AT -> C1206C475J3RACTU
- C10, C11, C12, C13, C14, C15, C16, C17, C4, C7, C8: Description CAP CER 0.1UF 16V X7R 0402 -> CAP CER 0.1UF 25V X7R 0402; Digikey PartNumber 490-6328-1-ND -> 478-10050-1-ND; Manufactured Part Number GRM155R71C104KA88J -> 04023C104JAT2A; Maufaturer Murata -> AVX Corporation
- R3, R4: Description RES SMD 0 OHM JUMPER 1/8W 0805 -> RES SMD 0 OHM JUMPER 1/16W 0402; Digikey PartNumber 541-0.0ACT-ND -> 541-0.0JCT-ND; Manufactured Part Number CRCW08050000Z0EA -> CRCW04020000Z0ED

Commit message: updated BOM
Parts:
- C1, C2, C5, C9: value 4.7uF -> 4.7UF,1206
- C10, C11, C12, C13, C14, C15, C16, C17, C4, C7, C8: value 0.1uF -> 0.1UF,0402
- C3, C6: value 18PF -> 18PF,0402
- D1, D2: value ~ -> CG0603MLC-12E; Description (none) -> VARISTOR 0603; Digikey PartNumber (none) -> CG0603MLC-12ECT-ND; Manufactured Part Number (none) -> CG0603MLC-12E; Maufaturer (none) -> Bourns Inc.
- FB1, FB2, FB3: value 600R -> 600E,FB,0402; Description FERRITE BEAD 600 OHM 0603 1LN -> FERRITE BEAD 600 OHM 0402 1LN; Digikey PartNumber 732-1593-1-ND -> 732-2388-1-ND; Manufactured Part Number 742792651 -> 7427927291; Maufaturer Würth Elektronik -> Wurth Elektronik
- J1: value Micro_USB -> 10118193-0001LF; Description (none) -> CONN RCPT USB2.0 MICRO B SMD R/A; Digikey PartNumber (none) -> 609-4616-2-ND; Manufactured Part Number (none) -> 10118193-0001LF; Maufaturer (none) -> Amphenol ICC (FCI)
- J2: Description (none) -> CONN HEADER VERT 8POS 2.54MM; Digikey PartNumber (none) -> 609-3264-ND; Manufactured Part Number (none) -> 68000-408HLF; Maufaturer (none) -> Amphenol ICC (FCI)
- J3: Description (none) -> CONN HEADER VERT 3POS 2.54MM; Digikey PartNumber (none) -> 609-3464-ND; Manufactured Part Number (none) -> 68000-203HLF; Maufaturer (none) -> Amphenol ICC (FCI)
- R1: value 1k -> 1KE,0402
- R10, R11, R12, R13, R14, R15, R16, R17, R18, R5, R6, R7, R8, R9: value 1K -> 1KE,0402
- R2: value 12K -> 12KE,0402
- R3, R4: value 0E -> 0E, 0402
- U1: Description Single chip USB to UART (RS232, RS422 or RS485) -> IC USB HS DUAL UART/FIFO 64-LQFP; Digikey PartNumber (none) -> 768-1024-1-ND; Manufactured Part Number (none) -> FT2232HL-REEL; Maufaturer (none) -> FTDI, Future Technology Devices International Ltd

Commit message: updated commented pending schematic
Parts:
- removed J1: 10118193-0001LF, symbol Aardonyx-rescue:USB_OTG-aardonyx
- added J1: USB_OTG, symbol Aardonyx-rescue:USB_OTG-skt32e_asic
Connections:
- no-connect marks 26 -> 30

Commit message: updated footprint for netlist
Parts:
- C1, C2, C5, C9: footprint (none) -> Capacitor_SMD:C_1206_3216Metric
- C10, C11, C12, C13, C14, C15, C16, C17, C3, C4, C6, C7, C8: footprint (none) -> Capacitor_SMD:C_0402_1005Metric
- D1, D2: footprint (none) -> Diode_SMD:D_0603_1608Metric
- FB1, FB2, FB3: footprint (none) -> Inductor_SMD:L_0603_1608Metric
- J3: footprint (none) -> Connector:FanPinHeader_1x03_P2.54mm_Vertical
- R1, R10, R11, R12, R13, R14, R15, R16, R17, R18, R2, R3, R4, R5, R6, R7, R8, R9: footprint (none) -> Resistor_SMD:R_0402_1005Metric
- TP1, TP2: footprint (none) -> TestPoint:TestPoint_Bridge_Pitch2.54mm_Drill0.7mm
- U1: footprint (none) -> Package_QFP:LQFP-64_10x10mm_P0.5mm
- Y1: footprint (none) -> Crystal:Crystal_SMD_HC49-SD_HandSoldering

Commit message: Updated schematic
Parts:
- removed J1: USB_OTG, symbol Aardonyx-rescue:USB_OTG-skt32e_asic
- added C91: 4.7UF,1206, Capacitor_SMD:C_1206_3216Metric, symbol Aardonyx-rescue:C_Small-aardonyx
- added C92: 0.1UF,0402, Capacitor_SMD:C_0402_1005Metric, symbol Aardonyx-rescue:C_Small-aardonyx
- added FB4, FB5: 600E,FB,0402, Inductor_SMD:L_0603_1608Metric, symbol Aardonyx-rescue:Ferrite_Bead_Small-aardonyx
- added J1: USB_B_6PIN, symbol Aardonyx-rescue:USB_B_6PIN
- added J17: USB_OTG, symbol Aardonyx-rescue:USB_OTG-aardonyx
- added J18: Conn_1x3_M, Connector:FanPinHeader_1x03_P2.54mm_Vertical, symbol Aardonyx-rescue:Conn_1x3_M-aardonyx
- added R38, R39: 22E,0402, Resistor_SMD:R_0402_1005Metric, symbol Aardonyx-rescue:R_US-aardonyx
- added R49: 0E, 0402, Resistor_SMD:R_0402_1005Metric, symbol Aardonyx-rescue:R_US-aardonyx
- added R50: 4.7KE,0402, Resistor_SMD:R_0402_1005Metric, symbol Aardonyx-rescue:R_US-aardonyx
- added R52: 10KE,0402, Resistor_SMD:R_0402_1005Metric, symbol Aardonyx-rescue:R_US-aardonyx
- added TP6: TestPoint, symbol Aardonyx-rescue:TestPoint-aardonyx
- added U16: 93LC56BT-I_OT, Package_TO_SOT_SMD:SOT-23-6, symbol Aardonyx-rescue:93LC56BT-I_OT
- C1, C2, C5, C9: Description CAP CER 4.7UF 25V X7R 1206 -> CAP TANT 4.7UF 10% 16V 1206; Digikey PartNumber 399-8203-1-ND -> 399-3697-1-ND; Manufactured Part Number C1206C475J3RACTU -> T491A475K016AT
- D1, D2: value CG0603MLC-12E -> CG0603MLC-12E
Connections:
- net labels added: GNDA, PWRSAV, RESET, USB_DM, USB_DP, VBUS_USB1, VBUS_USB2
- wire segments 212 -> 256
- no-connect marks 30 -> 26
Other:
- note added: "2Kb 16bit Serial EEPROM"
- note added: "64PIN LQFP"
- note added: "SOT23-6"
- note added: "Short 1 & 2, VBUS = VBUS_USB1\nShort 2 & 3, VBUS = VBUS_USB2"
- note added: "USB - JTAG/UART DUAL PORT CONVERTER\n"
- note added: "Use J1 for high loads"
- note added: "Use J17 for low \npower applications\n"
- note removed: "FTDI - USB TO JTAG/UART"
- moved on the sheet: C1, C11, C12, C13, C14, C15, C16, C17, D1, D2, FB1, J2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

Commit message: Update Footprint
Parts:
- J1, J17: footprint (none) -> Aardonyx:USB_2.0_Micro-B_AMPHENOL_HPL_510
- J2: footprint (none) -> Connector_PinHeader_2.54mm:PinHeader_1x08_P2.54mm_Vertical
- TP6: footprint (none) -> TestPoint:TestPoint_Bridge_Pitch2.54mm_Drill0.7mm
Changed lines of the file:
@@
 EESchema Schematic File Version 4
-LIBS:Aardonyx-cache
-EELAYER 29 0
+EELAYER 30 0
 EELAYER END
 $Descr A4 11693 8268
@@
 F 0 "J2" H 9050 3850 50  0000 L CNN
 F 1 "Conn_1x8" H 8950 2950 50  0000 L CNN
-F 2 "" H 9100 3450 50  0001 C CNN
+F 2 "Connector_PinHeader_2.54mm:PinHeader_1x08_P2.54mm_Vertical" H 9100 3450 50  0001 C CNN
 F 3 "https://www.digikey.com/products/en?keywords=68000-408HLF" H 9100 3450 50  0001 C CNN
 F 4 "CONN HEADER VERT 8POS 2.54MM" H 9100 3450 50  0001 C CNN "Description"
@@
 F 0 "J17" H 1500 4117 50  0000 C CNN
 F 1 "USB_OTG" H 1500 4026 50  0000 C CNN
-F 2 "" H 1750 3600 50  0001 C CNN
+F 2 "Aardonyx:USB_2.0_Micro-B_AMPHENOL_HPL_510" H 1750 3600 50  0001 C CNN
 F 3 "https://www.digikey.com/product-detail/en/amphenol-icc-fci/10118194-0001LF/609-4618-1-ND/2785382" H 1750 3600 50  0001 C CNN
 F 4 "CONN RCPT USB2.0 MICRO B SMD R/A" H 1600 3650 50  0001 C CNN "Description"
@@
 F 0 "J1" H 1203 2267 50  0000 C CNN
 F 1 "USB_B_6PIN" H 1203 2176 50  0000 C CNN
-F 2 "" H 1300 1750 50  0001 C CNN
+F 2 "Aardonyx:USB_2.0_Micro-B_AMPHENOL_HPL_510" H 1300 1750 50  0001 C CNN
 F 3 "https://www.digikey.com/product-detail/en/amphenol-icc-fci/61729-0010BLF/609-1039-ND/1001353" H 1300 1750 50  0001 C CNN
 F 4 "CONN RCPT USB2.0 TYPEB 4POS R/A" H 1150 1800 50  0001 C CNN "Description"
@@
 F 0 "TP6" V 3050 4750 50  0000 R CNN
 F 1 "TestPoint" V 3000 4950 50  0000 R CNN
-F 2 "" H 3250 4450 50  0001 C CNN
+F 2 "TestPoint:TestPoint_Bridge_Pitch2.54mm_Drill0.7mm" H 3250 4450 50  0001 C CNN
 F 3 "" H 3250 4450 50  0001 C CNN
 	1    3050 4450

Commit message: Updated footprint association
Parts:
- FB1, FB2, FB3, FB4, FB5: footprint Inductor_SMD:L_0603_1608Metric -> Inductor_SMD:L_0402_1005Metric
- J1: footprint Aardonyx:USB_2.0_Micro-B_AMPHENOL_HPL_510 -> Connector_USB:USB_B_OST_USB-B1HSxx_Horizontal
- J17: footprint Aardonyx:USB_2.0_Micro-B_AMPHENOL_HPL_510 -> Connector_USB:USB_Micro-B_Amphenol_10103594-0001LF_Horizontal
- J18, J3: footprint Connector:FanPinHeader_1x03_P2.54mm_Vertical -> Connector_PinHeader_2.54mm:PinHeader_1x03_P2.54mm_Vertical
Changed lines of the file:
@@
 EESchema Schematic File Version 4
-EELAYER 30 0
+LIBS:Aardonyx-cache
+EELAYER 29 0
 EELAYER END
 $Descr A4 11693 8268
@@
 F 0 "FB3" V 3413 1800 50  0000 C CNN
 F 1 "600E,FB,0402" V 3504 1800 50  0000 C CNN
-F 2 "Inductor_SMD:L_0603_1608Metric" V 3580 1800 50  0001 C CNN
+F 2 "Inductor_SMD:L_0402_1005Metric" V 3580 1800 50  0001 C CNN
 F 3 "https://www.digikey.in/product-detail/en/w%C3%BCrth-elektronik/742792651/732-1593-1-ND/1639537" H 3650 1800 50  0001 C CNN
 F 4 "FERRITE BEAD 600 OHM 0402 1LN" H 3650 1800 50  0001 C CNN "Description"
@@
 F 0 "FB2" V 3413 1350 50  0000 C CNN
 F 1 "600E,FB,0402" V 3504 1350 50  0000 C CNN
-F 2 "Inductor_SMD:L_0603_1608Metric" V 3580 1350 50  0001 C CNN
+F 2 "Inductor_SMD:L_0402_1005Metric" V 3580 1350 50  0001 C CNN
 F 3 "https://www.digikey.in/product-detail/en/w%C3%BCrth-elektronik/742792651/732-1593-1-ND/1639537" H 3650 1350 50  0001 C CNN
 F 4 "FERRITE BEAD 600 OHM 0402 1LN" H 3650 1350 50  0001 C CNN "Description"
@@
 F 0 "FB1" H 1900 2800 50  0000 C CNN
 F 1 "600E,FB,0402" V 2100 2900 50  0000 C CNN
-F 2 "Inductor_SMD:L_0603_1608Metric" V 1930 2900 50  0001 C CNN
+F 2 "Inductor_SMD:L_0402_1005Metric" V 1930 2900 50  0001 C CNN
 F 3 "https://www.digikey.in/product-detail/en/w%C3%BCrth-elektronik/742792651/732-1593-1-ND/1639537" H 2000 2900 50  0001 C CNN
 F 4 "FERRITE BEAD 600 OHM 0402 1LN" H 2000 2900 50  0001 C CNN "Description"
@@
 F 0 "J3" H 9300 5650 50  0000 L CNN
 F 1 "Conn_1x3_M" H 9200 5250 50  0000 L CNN
-F 2 "Connector:FanPinHeader_1x03_P2.54mm_Vertical" H 9300 5450 50  0001 C CNN
+F 2 "Connector_PinHeader_2.54mm:PinHeader_1x03_P2.54mm_Vertical" H 9300 5450 50  0001 C CNN
 F 3 "https://www.digikey.com/product-detail/en/amphenol-icc-fci/68000-203HLF/609-3464-ND/2023305" H 9300 5450 50  0001 C CNN
 F 4 "CONN HEADER VERT 3POS 2.54MM" H 9300 5450 50  0001 C CNN "Description"
@@
 F 0 "J17" H 1500 4117 50  0000 C CNN
 F 1 "USB_OTG" H 1500 4026 50  0000 C CNN
-F 2 "Aardonyx:USB_2.0_Micro-B_AMPHENOL_HPL_510" H 1750 3600 50  0001 C CNN
+F 2 "Connector_USB:USB_Micro-B_Amphenol_10103594-0001LF_Horizontal" H 1750 3600 50  0001 C CNN
 F 3 "https://www.digikey.com/product-detail/en/amphenol-icc-fci/10118194-0001LF/609-4618-1-ND/2785382" H 1750 3600 50  0001 C CNN
 F 4 "CONN RCPT USB2.0 MICRO B SMD R/A" H 1600 3650 50  0001 C CNN "Description"
@@
 F 0 "FB5" H 2300 6800 50  0000 C CNN
 F 1 "600E,FB,0402" V 2500 6900 50  0000 C CNN
-F 2 "Inductor_SMD:L_0603_1608Metric" V 2330 6900 50  0001 C CNN
+F 2 "Inductor_SMD:L_0402_1005Metric" V 2330 6900 50  0001 C CNN
 F 3 "https://www.digikey.in/product-detail/en/w%C3%BCrth-elektronik/742792651/732-1593-1-ND/1639537" H 2400 6900 50  0001 C CNN
 F 4 "FERRITE BEAD 600 OHM 0402 1LN" H 2400 6900 50  0001 C CNN "Description"
@@
 F 0 "J1" H 1203 2267 50  0000 C CNN
 F 1 "USB_B_6PIN" H 1203 2176 50  0000 C CNN
-F 2 "Aardonyx:USB_2.0_Micro-B_AMPHENOL_HPL_510" H 1300 1750 50  0001 C CNN
+F 2 "Connector_USB:USB_B_OST_USB-B1HSxx_Horizontal" H 1300 1750 50  0001 C CNN
 F 3 "https://www.digikey.com/product-detail/en/amphenol-icc-fci/61729-0010BLF/609-1039-ND/1001353" H 1300 1750 50  0001 C CNN
 F 4 "CONN RCPT USB2.0 TYPEB 4POS R/A" H 1150 1800 50  0001 C CNN "Description"
@@
 F 0 "FB4" H 1450 950 50  0000 C CNN
 F 1 "600E,FB,0402" V 1650 1050 50  0000 C CNN
-F 2 "Inductor_SMD:L_0603_1608Metric" V 1480 1050 50  0001 C CNN
+F 2 "Inductor_SMD:L_0402_1005Metric" V 1480 1050 50  0001 C CNN
 F 3 "https://www.digikey.in/product-detail/en/w%C3%BCrth-elektronik/742792651/732-1593-1-ND/1639537" H 1550 1050 50  0001 C CNN
 F 4 "FERRITE BEAD 600 OHM 0402 1LN" H 1550 1050 50  0001 C CNN "Description"
@@
 F 0 "J18" H 2950 1850 50  0000 L CNN
 F 1 "Conn_1x3_M" H 2600 1450 50  0000 L CNN
-F 2 "Connector:FanPinHeader_1x03_P2.54mm_Vertical" H 2950 1650 50  0001 C CNN
+F 2 "Connector_PinHeader_2.54mm:PinHeader_1x03_P2.54mm_Vertical" H 2950 1650 50  0001 C CNN
 F 3 "https://www.digikey.com/product-detail/en/amphenol-icc-fci/68000-203HLF/609-3464-ND/2023305" H 2950 1650 50  0001 C CNN
 F 4 "CONN HEADER VERT 3POS 2.54MM" H 2950 1650 50  0001 C CNN "Description"
