File: asic/e-class-aardonyx/board/Board_Design/power_1.sch (KiCad schematic (older format))
At the start: 38 parts, among them J8 12V, J9 Conn_1x3_M, SW1 SW_SPST, U10 TPS62086RLTR, U11 TPS54627DDAR, U9 TPS62061DSGR

Commit message: update
Parts:
- removed C63, C64, C70: 10UF, symbol aardonyx:C_Small
- removed C68: 22PF, symbol aardonyx:C_Small
- removed C69: 22UF, symbol aardonyx:C_Small
- removed L1: 1.0UH, symbol aardonyx:L
- removed L2: 0.47UH, symbol aardonyx:L
- removed R70: 360K, symbol aardonyx:R_US
- removed R71: 180K, symbol aardonyx:R_US
- removed U10: TPS62086RLTR, symbol aardonyx:TPS62086RLTR
- removed U9: TPS62061DSGR, symbol aardonyx:TPS62061DSGR
- gave numbers to parts that had none: 5
- renumbered C71 to C63, C72 to C64, C73 to C65, C74 to C66, C65 to C67, C66 to C68, C67 to C69, C75 to C70, C76 to C71, C77 to C73, C78 to C75, C79 to C76, J9 to J10, J8 to J9, L3 to L2, R72 to R85, R73 to R86, R74 to R87, R75 to R88, U11 to U9
Connections:
- net labels removed: V1P8, V3P3
- wire segments 149 -> 98
- no-connect marks 1 -> 0
Other:
- note removed: "SWITCHING REGULATOR FOR V1P8 POWER RAIL"
- note removed: "SWITCHING REGULATOR FOR V3P3 POWER RAIL"
- note removed: "VOLTAGE SEQUENCER"

Commit message: update
Parts:
- renumbered C63 to C33, C64 to C34, C65 to C35, C66 to C36, C67 to C37, C68 to C38, C69 to C39, C70 to C40, C71 to C41, C72 to C42, C73 to C43, C74 to C44, C75 to C45, C76 to C46, J9 to J3, J10 to J4, R85 to R25, R86 to R26, R87 to R27, R88 to R28, R89 to R29, U9 to U4

Commit message: update
Parts:
- renumbered J3 to J5, J4 to J6
Changed lines of the file:
@@
 encoding utf-8
 Sheet 4 7
-Title ""
+Title "AARDONYX_DEVELOPMENT_BOARD"
 Date ""
-Rev ""
-Comp ""
+Rev "R1V0"
+Comp "IIT_MADRAS"
 Comment1 ""
 Comment2 ""
@@
 Connection ~ 2250 4600
 $Comp
-L aardonyx:V12P0 #PWR033
+L aardonyx:V12P0 #PWR036
 U 1 1 5E79C895
 P 2250 4450
-AR Path="/5DB8A7DC/5E79C895" Ref="#PWR033"  Part="1"
+AR Path="/5DB8A7DC/5E79C895" Ref="#PWR036"  Part="1"
 AR Path="/5E6E93B2/5E79C895" Ref="#PWR?"  Part="1"
-F 0 "#PWR033" H 2400 4400 50  0001 C CNN
+F 0 "#PWR036" H 2400 4400 50  0001 C CNN
 F 1 "V12P0" H 2255 4625 50  0000 C CNN
 F 2 "" H 2250 4450 50  0001 C CNN
@@
 	8500 5500 8500 5800
 $Comp
-L aardonyx:GND #PWR046
+L aardonyx:GND #PWR049
 U 1 1 5DC268B2
 P 8500 5800
-AR Path="/5DB8A7DC/5DC268B2" Ref="#PWR046"  Part="1"
+AR Path="/5DB8A7DC/5DC268B2" Ref="#PWR049"  Part="1"
 AR Path="/5E6E93B2/5DC268B2" Ref="#PWR?"  Part="1"
-F 0 "#PWR046" H 8500 5550 50  0001 C CNN
+F 0 "#PWR049" H 8500 5550 50  0001 C CNN
 F 1 "GND" H 8505 5627 50  0000 C CNN
 F 2 "" H 8500 5800 50  0001 C CNN
@@
 Connection ~ 7250 5500
 $Comp
-L aardonyx:GND #PWR041
+L aardonyx:GND #PWR044
 U 1 1 5DC135E5
 P 7250 6100
-AR Path="/5DB8A7DC/5DC135E5" Ref="#PWR041"  Part="1"
+AR Path="/5DB8A7DC/5DC135E5" Ref="#PWR044"  Part="1"
 AR Path="/5E6E93B2/5DC135E5" Ref="#PWR?"  Part="1"
-F 0 "#PWR041" H 7250 5850 50  0001 C CNN
+F 0 "#PWR044" H 7250 5850 50  0001 C CNN
 F 1 "GND" H 7255 5927 50  0000 C CNN
 F 2 "" H 7250 6100 50  0001 C CNN
@@
 $EndComp
 $Comp
-L aardonyx:GND #PWR034
+L aardonyx:GND #PWR037
 U 1 1 5DC06DDF
 P 2250 5300
-AR Path="/5DB8A7DC/5DC06DDF" Ref="#PWR034"  Part="1"
+AR Path="/5DB8A7DC/5DC06DDF" Ref="#PWR037"  Part="1"
 AR Path="/5E6E93B2/5DC06DDF" Ref="#PWR?"  Part="1"
-F 0 "#PWR034" H 2250 5050 50  0001 C CNN
+F 0 "#PWR037" H 2250 5050 50  0001 C CNN
 F 1 "GND" H 2255 5127 50  0000 C CNN
 F 2 "" H 2250 5300 50  0001 C CNN
@@
 	4050 5200 4750 5200
 $Comp
-L aardonyx:GND #PWR036
+L aardonyx:GND #PWR039
 U 1 1 5DBFE03A
 P 4450 6100
-AR Path="/5DB8A7DC/5DBFE03A" Ref="#PWR036"  Part="1"
+AR Path="/5DB8A7DC/5DBFE03A" Ref="#PWR039"  Part="1"
 AR Path="/5E6E93B2/5DBFE03A" Ref="#PWR?"  Part="1"
-F 0 "#PWR036" H 4450 5850 50  0001 C CNN
+F 0 "#PWR039" H 4450 5850 50  0001 C CNN
 F 1 "GND" H 4455 5927 50  0000 C CNN
 F 2 "" H 4450 6100 50  0001 C CNN
@@
 $EndComp
 $Comp
-L aardonyx:GND #PWR037
+L aardonyx:GND #PWR040
 U 1 1 5DBF95B1
 P 5300 6100
-AR Path="/5DB8A7DC/5DBF95B1" Ref="#PWR037"  Part="1"
+AR Path="/5DB8A7DC/5DBF95B1" Ref="#PWR040"  Part="1"
 AR Path="/5E6E93B2/5DBF95B1" Ref="#PWR?"  Part="1"
-F 0 "#PWR037" H 5300 5850 50  0001 C CNN
+F 0 "#PWR040" H 5300 5850 50  0001 C CNN
 F 1 "GND" H 5305 5927 50  0000 C CNN
 F 2 "" H 5300 6100 50  0001 C CNN
@@
 $EndComp
 $Comp
-L aardonyx:V5P0 #PWR045
+L aardonyx:V5P0 #PWR048
 U 1 1 5DC202F3
 P 8150 4100
-AR Path="/5DB8A7DC/5DC202F3" Ref="#PWR045"  Part="1"
+AR Path="/5DB8A7DC/5DC202F3" Ref="#PWR048"  Part="1"
 AR Path="/5E6E93B2/5DC202F3" Ref="#PWR?"  Part="1"
-F 0 "#PWR045" H 8300 4050 50  0001 C CNN
+F 0 "#PWR048" H 8300 4050 50  0001 C CNN
 F 1 "V5P0" H 8145 4275 50  0000 C CNN
 F 2 "" H 8150 4100 50  0001 C CNN
@@
 $EndComp
 $Comp
-L aardonyx:Barrel_Jack_Switch J3
+L aardonyx:Barrel_Jack_Switch J5
 U 1 1 5E7997C5
 P 3400 1700
-AR Path="/5DB8A7DC/5E7997C5" Ref="J3"  Part="1"
+AR Path="/5DB8A7DC/5E7997C5" Ref="J5"  Part="1"
 AR Path="/5E6E93B2/5E7997C5" Ref="J?"  Part="1"
-F 0 "J3" H 3300 1900 50  0000 C CNN
+F 0 "J5" H 3300 1900 50  0000 C CNN
 F 1 "12V" H 3550 1500 50  0000 C CNN
 F 2 "" H 3450 1660 50  0001 C CNN
@@
 $EndComp
 $Comp
-L aardonyx:GND #PWR035
+L aardonyx:GND #PWR038
 U 1 1 5DC2CAAD
 P 3850 1950
-AR Path="/5DB8A7DC/5DC2CAAD" Ref="#PWR035"  Part="1"
+AR Path="/5DB8A7DC/5DC2CAAD" Ref="#PWR038"  Part="1"
 AR Path="/5E6E93B2/5DC2CAAD" Ref="#PWR?"  Part="1"
-F 0 "#PWR035" H 3850 1700 50  0001 C CNN
+F 0 "#PWR038" H 3850 1700 50  0001 C CNN
 F 1 "GND" H 3855 1777 50  0000 C CNN
 F 2 "" H 3850 1950 50  0001 C CNN
@@
 	5450 1600 5450 1750
 $Comp
-L aardonyx:V12P0 #PWR042
+L aardonyx:V12P0 #PWR045
 U 1 1 5E820603
 P 7750 1350
-AR Path="/5DB8A7DC/5E820603" Ref="#PWR042"  Part="1"
+AR Path="/5DB8A7DC/5E820603" Ref="#PWR045"  Part="1"
 AR Path="/5E6E93B2/5E820603" Ref="#PWR?"  Part="1"
-F 0 "#PWR042" H 7900 1300 50  0001 C CNN
+F 0 "#PWR045" H 7900 1300 50  0001 C CNN
 F 1 "V12P0" H 7755 1525 50  0000 C CNN
 F 2 "" H 7750 1350 50  0001 C CNN
@@
 	5450 1600 5800 1600
 $Comp
-L aardonyx:GND #PWR038
+L aardonyx:GND #PWR041
 U 1 1 5E83D54C
 P 5800 2200
-AR Path="/5DB8A7DC/5E83D54C" Ref="#PWR038"  Part="1"
+AR Path="/5DB8A7DC/5E83D54C" Ref="#PWR041"  Part="1"
 AR Path="/5E6E93B2/5E83D54C" Ref="#PWR?"  Part="1"
-F 0 "#PWR038" H 5800 1950 50  0001 C CNN
+F 0 "#PWR041" H 5800 1950 50  0001 C CNN
 F 1 "GND" H 5805 2027 50  0000 C CNN
 F 2 "" H 5800 2200 50  0001 C CNN
@@
 P 8750 4200
 AR Path="/5D8B37DE/5E52467C" Ref="J?"  Part="1"
-AR Path="/5DB8A7DC/5E52467C" Ref="J4"  Part="1"
+AR Path="/5DB8A7DC/5E52467C" Ref="J6"  Part="1"
 AR Path="/5E6E93B2/5E52467C" Ref="J?"  Part="1"
-F 0 "J4" H 8750 4400 50  0000 L CNN
+F 0 "J6" H 8750 4400 50  0000 L CNN
 F 1 "Conn_1x3_M" H 8650 4000 50  0000 L CNN
 F 2 "" H 8750 4200 50  0001 C CNN
@@
 Connection ~ 5100 1600
 $Comp
-L aardonyx:GND #PWR039
+L aardonyx:GND #PWR042
 U 1 1 5E5D54A0
 P 6200 2000
-AR Path="/5DB8A7DC/5E5D54A0" Ref="#PWR039"  Part="1"
+AR Path="/5DB8A7DC/5E5D54A0" Ref="#PWR042"  Part="1"
 AR Path="/5E6E93B2/5E5D54A0" Ref="#PWR?"  Part="1"
-F 0 "#PWR039" H 6200 1750 50  0001 C CNN
+F 0 "#PWR042" H 6200 1750 50  0001 C CNN
 F 1 "GND" H 6205 1827 50  0000 C CNN
 F 2 "" H 6200 2000 50  0001 C CNN
@@
 $EndComp
 $Comp
-L aardonyx:GND #PWR040
+L aardonyx:GND #PWR043
 U 1 1 5E5D9EFD
 P 7050 2000
-AR Path="/5DB8A7DC/5E5D9EFD" Ref="#PWR040"  Part="1"
+AR Path="/5DB8A7DC/5E5D9EFD" Ref="#PWR043"  Part="1"
 AR Path="/5E6E93B2/5E5D9EFD" Ref="#PWR?"  Part="1"
-F 0 "#PWR040" H 7050 1750 50  0001 C CNN
+F 0 "#PWR043" H 7050 1750 50  0001 C CNN
 F 1 "GND" H 7055 1827 50  0000 C CNN
 F 2 "" H 7050 2000 50  0001 C CNN
@@
 	7750 1950 7750 2150
 $Comp
-L aardonyx:GND #PWR043
+L aardonyx:GND #PWR046
 U 1 1 5E5FEB09
 P 7750 2200
-AR Path="/5DB8A7DC/5E5FEB09" Ref="#PWR043"  Part="1"
+AR Path="/5DB8A7DC/5E5FEB09" Ref="#PWR046"  Part="1"
 AR Path="/5E6E93B2/5E5FEB09" Ref="#PWR?"  Part="1"
-F 0 "#PWR043" H 7750 1950 50  0001 C CNN
+F 0 "#PWR046" H 7750 1950 50  0001 C CNN
 F 1 "GND" H 7755 2027 50  0000 C CNN
 F 2 "" H 7750 2200 50  0001 C CNN
@@
 $EndComp
 $Comp
-L aardonyx:V5P0 #PWR047
+L aardonyx:V5P0 #PWR050
 U 1 1 5E699359
 P 10000 4450
-AR Path="/5DB8A7DC/5E699359" Ref="#PWR047"  Part="1"
+AR Path="/5DB8A7DC/5E699359" Ref="#PWR050"  Part="1"
 AR Path="/5E6E93B2/5E699359" Ref="#PWR?"  Part="1"
-F 0 "#PWR047" H 10150 4400 50  0001 C CNN
+F 0 "#PWR050" H 10150 4400 50  0001 C CNN
 F 1 "V5P0" H 9995 4625 50  0000 C CNN
 F 2 "" H 10000 4450 50  0001 C CNN
@@
 $EndComp
 $Comp
-L aardonyx:GND #PWR048
+L aardonyx:GND #PWR051
 U 1 1 5E69E227
 P 10000 5550
-AR Path="/5DB8A7DC/5E69E227" Ref="#PWR048"  Part="1"
+AR Path="/5DB8A7DC/5E69E227" Ref="#PWR051"  Part="1"
 AR Path="/5E6E93B2/5E69E227" Ref="#PWR?"  Part="1"
-F 0 "#PWR048" H 10000 5300 50  0001 C CNN
+F 0 "#PWR051" H 10000 5300 50  0001 C CNN
 F 1 "GND" H 10005 5377 50  0000 C CNN
 F 2 "" H 10000 5550 50  0001 C CNN
@@
 P 7950 4250
 AR Path="/5D8B3761/5E51F41F" Ref="#PWR?"  Part="1"
-AR Path="/5DB8A7DC/5E51F41F" Ref="#PWR044"  Part="1"
+AR Path="/5DB8A7DC/5E51F41F" Ref="#PWR047"  Part="1"
 AR Path="/5E6E93B2/5E51F41F" Ref="#PWR?"  Part="1"
-F 0 "#PWR044" H 8100 4200 50  0001 C CNN
+F 0 "#PWR047" H 8100 4200 50  0001 C CNN
 F 1 "VBUS" H 7955 4425 50  0000 C CNN
 F 2 "" H 7950 4250 50  0001 C CNN

Commit message: updare
Parts:
- R26: Field4 (none) -> NA
Changed lines of the file:
@@
 F 2 "" V 3790 5340 50  0001 C CNN
 F 3 "~" H 3750 5350 50  0001 C CNN
+F 4 "NA" H 3600 5350 50  0000 C CNN "Field4"
 	1    3750 5350
 	1    0    0    -1
