File: asic/e-class-aardonyx/board/Board_Design/power_1.sch (KiCad schematic (older format))
At the start: 27 parts, among them J5 12V, J6 Conn_1x3_M, SW1 SW_SPST, U4 TPS54627DDAR

Commit message: update bom
Parts:
- F1: Description (none) -> PTC RESET FUSE 30V 920MA RADIAL; Digikey PartNumber (none) -> BC2323-ND; Manufactured Part Number (none) -> PTCCL13H921DBE; Maufaturer (none) -> Vishay BC Components
- U4: Description (none) -> IC REG BUCK ADJUSTABLE 6A 8SOPWR; Digikey PartNumber (none) -> 296-40808-1-ND; Manufactured Part Number (none) -> TPS54627DDAR; Maufaturer (none) -> Texas Instruments
Changed lines of the file:
@@
 F 1 "TPS54627DDAR" H 5300 5724 50  0000 C CNN
 F 2 "" H 5300 5000 50  0001 C CNN
-F 3 "" H 5300 5000 50  0001 C CNN
+F 3 "https://www.digikey.in/product-detail/en/texas-instruments/TPS54627DDAR/296-40808-1-ND/5178685" H 5300 5000 50  0001 C CNN
+F 4 "IC REG BUCK ADJUSTABLE 6A 8SOPWR" H 5300 5050 50  0001 C CNN "Description"
+F 5 "296-40808-1-ND" H 5300 5050 50  0001 C CNN "Digikey PartNumber"
+F 6 "TPS54627DDAR" H 5300 5050 50  0001 C CNN "Manufactured Part Number"
+F 7 "Texas Instruments" H 5300 5050 50  0001 C CNN "Maufaturer"
 	1    5300 5050
 	1    0    0    -1
@@
 F 1 "PTCCL13H921DBE" V 4850 1600 50  0000 C CNN
 F 2 "" H 4750 1400 50  0001 L CNN
-F 3 "~" H 4700 1600 50  0001 C CNN
+F 3 "https://www.digikey.in/products/en?keywords=PTCCL13H921DBE" H 4700 1600 50  0001 C CNN
+F 4 "PTC RESET FUSE 30V 920MA RADIAL" H 4700 1600 50  0001 C CNN "Description"
+F 5 "BC2323-ND" H 4700 1600 50  0001 C CNN "Digikey PartNumber"
+F 6 "PTCCL13H921DBE" H 4700 1600 50  0001 C CNN "Manufactured Part Number"
+F 7 "Vishay BC Components" H 4700 1600 50  0001 C CNN "Maufaturer"
 	1    4700 1600
 	0    1    1    0

Commit message: update BOM
Parts:
- C33, C43, C45: Description CAP CER 22UF 16V X6S 1206 -> CAP CER 22UF 25V X5R 1206; Digikey PartNumber 490-12409-1-ND -> 1276-3047-1-ND; Manufactured Part Number GRT31CC81C226KE01L -> CL31A226KAHNNNE; Maufaturer Murata -> Samsung Electro-Mechanics
- C34, C39, C40, C44, C46: Description CAP CER 0.1UF 16V X7R 0402 -> CAP CER 0.1UF 25V X7R 0402; Digikey PartNumber 490-6328-1-ND -> 478-10050-1-ND; Manufactured Part Number GRM155R71C104KA88J -> 04023C104JAT2A; Maufaturer Murata -> AVX Corporation
- C35, C38, C42: Description CAP CER 1UF 16V Y5V 0805 -> CAP CER 1UF 25V X7R 0805; Digikey PartNumber 399-8011-1-ND -> 399-10060-6-ND; Manufactured Part Number 399-8011-1-ND -> C0805C105J3RACTU
- C37: Description (none) -> CAP TANT 220UF 20% 25V 3226; Digikey PartNumber (none) -> 718-1945-1-ND; Manufactured Part Number (none) -> 597D227X0025M2T; Maufaturer (none) -> Vishay Sprague
- C41: Description CAP CER 15PF 16V C0G/NP0 0402 -> CAP CER 15PF 25V C0G/NP0 0805; Digikey PartNumber 399-8947-1-ND -> 732-7828-1-ND; Manufactured Part Number C0402C150J4GACTU -> 885012007029; Maufaturer Kemet -> Würth Elektronik
- renumbered R25 to P_R25, R26 to P_R26, R27 to P_R27, R28 to P_R28, R29 to R29_0805

Commit message: updated BOM
Parts:
- C33, C43, C45: value 22UF -> 22UF,1206
- C34, C39, C40, C44, C46: value 0.1UF -> 0.1UF,0402
- C35, C38, C42: value 1UF -> 1UF,0805
- C36: value 7500PF -> 7500PF,0603
- C37: value 220UF -> 220UF,3226
- C41: value 15PF -> 15PF,0805; Maufaturer Würth Elektronik -> Wurth Elektronik
- D3: value LED_ALT -> LED,0603; Description (none) -> LED GREEN CLEAR CHIP SMD; Digikey PartNumber (none) -> 160-1832-1-ND; Manufactured Part Number (none) -> LTST-C193TGKT-5A; Maufaturer (none) -> Lite-On Inc.
- J5: Description (none) -> CONN PWR JACK 2X5.5MM KINKED PIN; Digikey PartNumber (none) -> CP-202AH-ND; Manufactured Part Number (none) -> PJ-202AH; Maufaturer (none) -> CUI Devices
- J6: Description (none) -> CONN HEADER VERT 3POS 2.54MM; Digikey PartNumber (none) -> 609-3464-ND; Manufactured Part Number (none) -> 68000-203HLF; Maufaturer (none) -> Amphenol ICC (FCI)
- L1: Description (none) -> CMC 15A 2LN 60 OHM SMD; Digikey PartNumber (none) -> 240-2501-1-ND; Manufactured Part Number (none) -> CM3421Y600R-10; Maufaturer (none) -> Laird-Signal Integrity Products
- L2: Description (none) -> FIXED IND 3.3UH 6.6A 17 MOHM SMD; Digikey PartNumber (none) -> 732-6781-2-ND; Manufactured Part Number (none) -> 78477033; Maufaturer (none) -> Wurth Elektronik
- P_R25, P_R26: value 10K -> 10KE,0805
- P_R27: value 124K -> 124KE,0805
- P_R28: value 22.1K -> 22.1KE,0805
- R29_805: renamed from R29_0805; value 1K -> 1KE,0402
- SW1: Description (none) -> SWITCH TOGGLE SPST 3A 120V; Digikey PartNumber (none) -> 450-2109-ND; Manufactured Part Number (none) -> TMS6T1B1M1QE; Maufaturer (none) -> TE Connectivity ALCOSWITCH Switches

Commit message: updated commented pending schematic
Parts:
- removed J5: 12V, symbol Aardonyx-rescue:Barrel_Jack_Switch-aardonyx
- removed P_R28: 22.1KE,0805, symbol Aardonyx-rescue:R_US-aardonyx
- removed SW1: SW_SPST, symbol Aardonyx-rescue:SW_SPST-aardonyx
- added J5: 12V, symbol Connector:Barrel_Jack_Switch
- added R27: 22.1KE,0805, symbol Aardonyx-rescue:R_US-skt32e_asic
- added SW1: SW_SPST, symbol Switch:SW_SPST
- renumbered P_R27 to R28, R29_805 to R29

Commit message: updated footprint for netlist
Parts:
- C33, C43, C45: footprint (none) -> Capacitor_SMD:C_1206_3216Metric
- C34, C39, C40, C44, C46: footprint (none) -> Capacitor_SMD:C_0402_1005Metric
- C35, C38, C41, C42: footprint (none) -> Capacitor_SMD:C_0805_2012Metric
- C36: footprint (none) -> Capacitor_SMD:C_0603_1608Metric
- D3: footprint (none) -> LED_SMD:LED_0603_1608Metric
- F1: footprint (none) -> Capacitor_THT:C_Disc_D9.0mm_W5.0mm_P7.50mm
- J6: footprint (none) -> Connector:FanPinHeader_1x03_P2.54mm_Vertical
- P_R25, P_R26, R27, R28: footprint (none) -> Resistor_SMD:R_0805_2012Metric
- R29: footprint (none) -> Resistor_SMD:R_0402_1005Metric
- U4: footprint (none) -> Package_SO:SOIC-8-1EP_3.9x4.9mm_P1.27mm_EP2.29x3mm_ThermalVias
Changed lines of the file:
@@
 EESchema Schematic File Version 4
-LIBS:Aardonyx-cache
-EELAYER 29 0
+EELAYER 30 0
 EELAYER END
 $Descr A4 11693 8268
@@
 F 0 "C46" H 8500 5300 50  0000 L CNN
 F 1 "0.1UF,0402" V 8550 4750 50  0000 L CNN
-F 2 "" H 8500 5200 50  0001 C CNN
+F 2 "Capacitor_SMD:C_0402_1005Metric" H 8500 5200 50  0001 C CNN
 F 3 "https://www.digikey.in/product-detail/en/avx-corporation/04023C104JAT2A/478-10050-1-ND/6564273" H 8500 5200 50  0001 C CNN
 F 4 "CAP CER 0.1UF 25V X7R 0402" H 8500 5200 50  0001 C CNN "Description"
@@
 F 0 "C45" H 8100 5300 50  0000 L CNN
 F 1 "22UF,1206" V 8200 4800 50  0000 L CNN
-F 2 "" H 8100 5200 50  0001 C CNN
+F 2 "Capacitor_SMD:C_1206_3216Metric" H 8100 5200 50  0001 C CNN
 F 3 "https://www.digikey.in/product-detail/en/samsung-electro-mechanics/CL31A226KAHNNNE/1276-3047-1-ND/3891133" H 8100 5200 50  0001 C CNN
 F 4 "CAP CER 22UF 25V X5R 1206" H 8100 5200 50  0001 C CNN "Description"
@@
 F 0 "C43" H 7700 5300 50  0000 L CNN
 F 1 "22UF,1206" V 7750 4750 50  0000 L CNN
-F 2 "" H 7700 5200 50  0001 C CNN
+F 2 "Capacitor_SMD:C_1206_3216Metric" H 7700 5200 50  0001 C CNN
 F 3 "https://www.digikey.in/product-detail/en/samsung-electro-mechanics/CL31A226KAHNNNE/1276-3047-1-ND/3891133" H 7700 5200 50  0001 C CNN
 F 4 "CAP CER 22UF 25V X5R 1206" H 7700 5200 50  0001 C CNN "Description"
@@
 F 0 "C41" H 6992 5246 50  0000 L CNN
 F 1 "15PF,0805" V 6850 4750 50  0000 L CNN
-F 2 "" H 6900 5200 50  0001 C CNN
+F 2 "Capacitor_SMD:C_0805_2012Metric" H 6900 5200 50  0001 C CNN
 F 3 "https://www.digikey.in/product-detail/en/w%C3%BCrth-elektronik/885012007029/732-7828-1-ND/5454455" H 6900 5200 50  0001 C CNN
 F 4 "CAP CER 15PF 25V C0G/NP0 0805" H 6900 5200 50  0001 C CNN "Description"
@@
 F 0 "C40" H 6050 4850 50  0000 L CNN
 F 1 "0.1UF,0402" H 6200 4700 50  0000 L CNN
-F 2 "" H 6200 4750 50  0001 C CNN
+F 2 "Capacitor_SMD:C_0402_1005Metric" H 6200 4750 50  0001 C CNN
 F 3 "https://www.digikey.in/product-detail/en/avx-corporation/04023C104JAT2A/478-10050-1-ND/6564273" H 6200 4750 50  0001 C CNN
 F 4 "CAP CER 0.1UF 25V X7R 0402" H 6200 4750 50  0001 C CNN "Description"
@@
 F 0 "C33" H 2100 4950 50  0000 L CNN
 F 1 "22UF,1206" V 2400 4600 50  0000 L CNN
-F 2 "" H 2250 4850 50  0001 C CNN
+F 2 "Capacitor_SMD:C_1206_3216Metric" H 2250 4850 50  0001 C CNN
 F 3 "https://www.digikey.in/product-detail/en/samsung-electro-mechanics/CL31A226KAHNNNE/1276-3047-1-ND/3891133" H 2250 4850 50  0001 C CNN
 F 4 "CAP CER 22UF 25V X5R 1206" H 2250 4850 50  0001 C CNN "Description"
@@
 F 0 "C34" H 2750 4950 50  0000 L CNN
 F 1 "0.1UF,0402" V 2800 4350 50  0000 L CNN
-F 2 "" H 2750 4850 50  0001 C CNN
+F 2 "Capacitor_SMD:C_0402_1005Metric" H 2750 4850 50  0001 C CNN
 F 3 "https://www.digikey.in/product-detail/en/avx-corporation/04023C104JAT2A/478-10050-1-ND/6564273" H 2750 4850 50  0001 C CNN
 F 4 "CAP CER 0.1UF 25V X7R 0402" H 2750 4850 50  0001 C CNN "Description"
@@
 F 0 "P_R25" V 3600 4750 50  0000 L CNN
 F 1 "10KE,0805" V 3400 4850 50  0000 L CNN
-F 2 "" V 3540 4890 50  0001 C CNN
+F 2 "Resistor_SMD:R_0805_2012Metric" V 3540 4890 50  0001 C CNN
 F 3 "https://www.digikey.in/product-detail/en/yageo/RC0805FR-0710KL/311-10-0KCRCT-ND/730482" H 3500 4900 50  0001 C CNN
 F 4 "RES SMD 10K OHM 1% 1/8W 0805" H 3500 4900 50  0001 C CNN "Description"
@@
 F 0 "P_R26" H 3818 5396 50  0000 L CNN
 F 1 "10KE,0805" H 3818 5305 50  0000 L CNN
-F 2 "" V 3790 5340 50  0001 C CNN
+F 2 "Resistor_SMD:R_0805_2012Metric" V 3790 5340 50  0001 C CNN
 F 3 "https://www.digikey.in/product-detail/en/yageo/RC0805FR-0710KL/311-10-0KCRCT-ND/730482" H 3750 5350 50  0001 C CNN
 F 4 "NA" H 3600 5350 50  0000 C CNN "Field4"
@@
 F 0 "C35" H 4050 5800 50  0000 L CNN
 F 1 "1UF,0805" V 4000 5300 50  0000 L CNN
-F 2 "" H 4050 5700 50  0001 C CNN
+F 2 "Capacitor_SMD:C_0805_2012Metric" H 4050 5700 50  0001 C CNN
 F 3 "https://www.digikey.in/product-detail/en/kemet/C0805C105J3RACTU/399-10060-6-ND/3739580" H 4050 5700 50  0001 C CNN
 F 4 "CAP CER 1UF 25V X7R 0805" H 4050 5700 50  0001 C CNN "Description"
@@
 F 0 "C36" H 4450 5800 50  0000 L CNN
 F 1 "7500PF,0603" V 4600 5200 50  0000 L CNN
-F 2 "" H 4450 5700 50  0001 C CNN
+F 2 "Capacitor_SMD:C_0603_1608Metric" H 4450 5700 50  0001 C CNN
 F 3 "https://www.digikey.in/product-detail/en/kemet/C0603C752J3GAC7867/399-9980-1-ND/3736979" H 4450 5700 50  0001 C CNN
 F 4 "CAP CER 7500PF 25V C0G/NP0 0603" H 4450 5700 50  0001 C CNN "Description"
@@
 F 0 "U4" H 5300 5815 50  0000 C CNN
 F 1 "TPS54627DDAR" H 5300 5724 50  0000 C CNN
-F 2 "" H 5300 5000 50  0001 C CNN
+F 2 "Package_SO:SOIC-8-1EP_3.9x4.9mm_P1.27mm_EP2.29x3mm_ThermalVias" H 5300 5000 50  0001 C CNN
 F 3 "https://www.digikey.in/product-detail/en/texas-instruments/TPS54627DDAR/296-40808-1-ND/5178685" H 5300 5000 50  0001 C CNN
 F 4 "IC REG BUCK ADJUSTABLE 6A 8SOPWR" H 5300 5050 50  0001 C CNN "Description"
@@
 F 0 "C38" H 5450 1950 50  0000 L CNN
 F 1 "1UF,0805" V 5550 1500 50  0000 L CNN
-F 2 "" H 5450 1850 50  0001 C CNN
+F 2 "Capacitor_SMD:C_0805_2012Metric" H 5450 1850 50  0001 C CNN
 F 3 "https://www.digikey.in/product-detail/en/kemet/C0805C105J3RACTU/399-10060-6-ND/3739580" H 5450 1850 50  0001 C CNN
 F 4 "CAP CER 1UF 25V X7R 0805" H 5450 1850 50  0001 C CNN "Description"
@@
 F 0 "C39" H 5800 1950 50  0000 L CNN
 F 1 "0.1UF,0402" V 5900 1450 50  0000 L CNN
-F 2 "" H 5800 1850 50  0001 C CNN
+F 2 "Capacitor_SMD:C_0402_1005Metric" H 5800 1850 50  0001 C CNN
 F 3 "https://www.digikey.in/product-detail/en/avx-corporation/04023C104JAT2A/478-10050-1-ND/6564273" H 5800 1850 50  0001 C CNN
 F 4 "CAP CER 0.1UF 25V X7R 0402" H 5800 1850 50  0001 C CNN "Description"
@@
 F 0 "J6" H 8750 4400 50  0000 L CNN
 F 1 "Conn_1x3_M" H 8650 4000 50  0000 L CNN
-F 2 "" H 8750 4200 50  0001 C CNN
+F 2 "Connector:FanPinHeader_1x03_P2.54mm_Vertical" H 8750 4200 50  0001 C CNN
 F 3 "https://www.digikey.com/product-detail/en/amphenol-icc-fci/68000-203HLF/609-3464-ND/2023305" H 8750 4200 50  0001 C CNN
 F 4 "CONN HEADER VERT 3POS 2.54MM" H 8750 4200 50  0001 C CNN "Description"
@@
 F 0 "C42" H 7400 1950 50  0000 L CNN
 F 1 "1UF,0805" V 7350 1450 50  0000 L CNN
-F 2 "" H 7400 1850 50  0001 C CNN
+F 2 "Capacitor_SMD:C_0805_2012Metric" H 7400 1850 50  0001 C CNN
 F 3 "https://www.digikey.in/product-detail/en/kemet/C0805C105J3RACTU/399-10060-6-ND/3739580" H 7400 1850 50  0001 C CNN
 F 4 "CAP CER 1UF 25V X7R 0805" H 7400 1850 50  0001 C CNN "Description"
@@
 F 0 "C44" H 7750 1950 50  0000 L CNN
 F 1 "0.1UF,0402" V 7950 1550 50  0000 L CNN
-F 2 "" H 7750 1850 50  0001 C CNN
+F 2 "Capacitor_SMD:C_0402_1005Metric" H 7750 1850 50  0001 C CNN
 F 3 "https://www.digikey.in/product-detail/en/avx-corporation/04023C104JAT2A/478-10050-1-ND/6564273" H 7750 1850 50  0001 C CNN
 F 4 "CAP CER 0.1UF 25V X7R 0402" H 7750 1850 50  0001 C CNN "Description"
@@
 F 0 "D3" V 10100 5100 50  0000 R CNN
 F 1 "LED,0603" V 9750 5100 50  0000 R CNN
-F 2 "" H 10000 5150 50  0001 C CNN
+F 2 "LED_SMD:LED_0603_1608Metric" H 10000 5150 50  0001 C CNN
 F 3 "https://www.digikey.com/product-detail/en/lite-on-inc/LTST-C193TGKT-5A/160-1832-1-ND/2356255" H 10000 5150 50  0001 C CNN
 F 4 "LED GREEN CLEAR CHIP SMD" H 10000 5150 50  0001 C CNN "Description"
@@
 F 0 "R29" H 10050 4800 50  0000 L CNN
 F 1 "1KE,0402" V 9900 4450 50  0000 L CNN
-F 2 "" V 10040 4690 50  0001 C CNN
+F 2 "Resistor_SMD:R_0402_1005Metric" V 10040 4690 50  0001 C CNN
 F 3 "https://www.digikey.in/product-detail/en/panasonic-electronic-components/ERJ-2GEJ102X/P1-0KJCT-ND/146897" H 10000 4700 50  0001 C CNN
 F 4 "RES SMD 1K OHM 5% 1/10W 0402" H 10000 4700 50  0001 C CNN "Description"
@@
 F 0 "R28" H 7318 5246 50  0000 L CNN
 F 1 "124KE,0805" V 7350 4750 50  0000 L CNN
-F 2 "" V 7290 5190 50  0001 C CNN
+F 2 "Resistor_SMD:R_0805_2012Metric" V 7290 5190 50  0001 C CNN
 F 3 "https://www.digikey.in/product-detail/en/panasonic-electronic-components/ERJ-6ENF1243V/P124KCCT-ND/119578" H 7250 5200 50  0001 C CNN
 F 4 "RES SMD 124K OHM 1% 1/8W 0805" H 7250 5200 50  0001 C CNN "Description"
@@
 F 0 "R27" H 7318 5846 50  0000 L CNN
 F 1 "22.1KE,0805" H 7318 5755 50  0000 L CNN
-F 2 "" V 7290 5790 50  0001 C CNN
+F 2 "Resistor_SMD:R_0805_2012Metric" V 7290 5790 50  0001 C CNN
 F 3 "https://www.digikey.in/product-detail/en/panasonic-electronic-components/ERA-6AEB2212V/P22-1KDACT-ND/3075024" H 7250 5800 50  0001 C CNN
 F 4 "https://www.digikey.in/product-detail/en/panasonic-electronic-components/ERA-6AEB2212V/P22-1KDACT-ND/3075024" H 7250 5800 50  0001 C CNN "Description"
@@
 F 0 "F1" V 4475 1600 50  0000 C CNN
 F 1 "PTCCL13H921DBE" V 4566 1600 50  0000 C CNN
-F 2 "" H 4750 1400 50  0001 L CNN
+F 2 "Capacitor_THT:C_Disc_D9.0mm_W5.0mm_P7.50mm" H 4750 1400 50  0001 L CNN
 F 3 "https://www.digikey.in/products/en?keywords=PTCCL13H921DBE" H 4700 1600 50  0001 C CNN
 F 4 "PTC RESET FUSE 30V 920MA RADIAL" H 4700 1600 50  0001 C CNN "Description"

Commit message: Updated schematic
Parts:
- removed SW1: SW_SPST, symbol Switch:SW_SPST
- added SW1: SW_SPST, symbol Aardonyx-rescue:SW_SPST
- added TP5: TestPoint, symbol Aardonyx-rescue:TestPoint-aardonyx
- C37: value 220UF,3226 -> 220UF,2924; Description CAP TANT 220UF 20% 25V 3226 -> CAP TANT POLY 220UF 25V 2924; Digikey PartNumber 718-1945-1-ND -> 478-12518-1-ND; Manufactured Part Number 597D227X0025M2T -> TCN4227M025R0100; Maufaturer Vishay Sprague -> AVX Corporation
- D3: value LED,0603 -> LED,1206; Description LED GREEN CLEAR CHIP SMD -> LED GREEN DIFFUSED 1206 SMD; Digikey PartNumber 160-1832-1-ND -> 67-1002-1-ND; Manufactured Part Number LTST-C193TGKT-5A -> SML-LX1206GW-TR; Maufaturer Lite-On Inc. -> Lumex Opto/Components Inc.
- J5: value 12V -> PJ-202H PWRJACK
- R27: Description https://www.digikey.in/product-detail/en/panasonic-electron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 -> RES 22.1K OHM 0.1% 1/8W 0805; Digikey PartNumber https://www.digikey.in/product-detail/en/panasonic-electron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 -> P22.1KDACT-ND; Manufactured Part Number https://www.digikey.in/product-detail/en/panasonic-electron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 -> ERA-6AEB2212V; Maufaturer https://www.digikey.in/product-detail/en/panasonic-electron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 -> Panasonic Electronic Components
Connections:
- net labels added: VCC5V
- wire segments 98 -> 99
Other:
- note added: "12V Power Input and protection\n"
- note added: "12V to 5V conversion using Switcher"
- note added: "Short 1 & 2, 5V from 12V to 5V converter\nShort 2 & 3, 5V from USB"
- note removed: "DC JACK POWER SUPPLY\n"
- note removed: "SWITCHING REGULATOR FOR V5P0 POWER RAIL"

Commit message: Update Footprint
Parts:
- C37: footprint (none) -> Aardonyx:CP_EIA-7260-38_VISHAY_Pad2.68x7.50mm_HandSolder
- J5: footprint (none) -> Aardonyx:Pwr_Jack_DC_PJ-202AH_Horizontal
- L1: footprint (none) -> Aardonyx:L_Laird_L9.55_W2.84
- L2: footprint (none) -> Aardonyx:L_Wuerth_WE_PDA_SMT-1280
- SW1: footprint (none) -> Button_Switch_THT:SW_NKK_G1xJP
- TP5: footprint (none) -> TestPoint:TestPoint_Bridge_Pitch2.54mm_Drill0.7mm
Changed lines of the file:
@@
 EESchema Schematic File Version 4
-LIBS:Aardonyx-cache
-EELAYER 29 0
+EELAYER 30 0
 EELAYER END
 $Descr A4 11693 8268
@@
 F 0 "L2" V 6700 5050 50  0000 C CNN
 F 1 "3.3UH" V 6600 4900 50  0000 C CNN
-F 2 "" H 6650 4900 50  0001 C CNN
+F 2 "Aardonyx:L_Wuerth_WE_PDA_SMT-1280" H 6650 4900 50  0001 C CNN
 F 3 "https://www.digikey.com/product-detail/en/w%C3%BCrth-elektronik/78477033/732-6781-2-ND/5168775" H 6650 4900 50  0001 C CNN
 F 4 "FIXED IND 3.3UH 6.6A 17 MOHM SMD" H 6650 4900 50  0001 C CNN "Description"
@@
 F 0 "C37" H 5100 1950 50  0000 L CNN
 F 1 "220UF,2924" V 5050 1350 50  0000 L CNN
-F 2 "" H 5100 1850 50  0001 C CNN
+F 2 "Aardonyx:CP_EIA-7260-38_VISHAY_Pad2.68x7.50mm_HandSolder" H 5100 1850 50  0001 C CNN
 F 3 "https://www.digikey.com/product-detail/en/avx-corporation/TCN4227M025R0100/478-12518-1-ND/9836495" H 5100 1850 50  0001 C CNN
 F 4 "CAP TANT POLY 220UF 25V 2924" H 5100 1850 50  0001 C CNN "Description"
@@
 F 0 "L1" H 6600 1981 50  0000 C CNN
 F 1 "CM3421Y600R-10" H 6600 1550 50  0000 C CNN
-F 2 "" H 6600 1700 50  0001 C CNN
+F 2 "Aardonyx:L_Laird_L9.55_W2.84" H 6600 1700 50  0001 C CNN
 F 3 "https://www.digikey.com/product-detail/en/laird-signal-integrity-products/CM3421Y600R-10/240-2501-1-ND/935987" H 6600 1700 50  0001 C CNN
 F 4 "	CMC 15A 2LN 60 OHM SMD" H 6600 1700 50  0001 C CNN "Description"
@@
 F 0 "J5" H 3457 2017 50  0000 C CNN
 F 1 "PJ-202H PWRJACK" H 3450 1500 50  0000 C CNN
-F 2 "" H 3450 1660 50  0001 C CNN
+F 2 "Aardonyx:Pwr_Jack_DC_PJ-202AH_Horizontal" H 3450 1660 50  0001 C CNN
 F 3 "https://www.digikey.com/products/en?keywords=PJ-202AH" H 3450 1660 50  0001 C CNN
 F 4 "CONN PWR JACK 2X5.5MM KINKED PIN" H 3400 1700 50  0001 C CNN "Description"
@@
 F 0 "TP5" V 10104 6238 50  0000 L CNN
 F 1 "TestPoint" V 10195 6238 50  0000 L CNN
-F 2 "" H 10350 6050 50  0001 C CNN
+F 2 "TestPoint:TestPoint_Bridge_Pitch2.54mm_Drill0.7mm" H 10350 6050 50  0001 C CNN
 F 3 "" H 10350 6050 50  0001 C CNN
 	1    10150 6050
@@
 F 0 "SW1" H 4200 1835 50  0000 C CNN
 F 1 "SW_SPST" H 4200 1744 50  0000 C CNN
-F 2 "" H 4200 1600 50  0001 C CNN
+F 2 "Button_Switch_THT:SW_NKK_G1xJP" H 4200 1600 50  0001 C CNN
 F 3 "https://www.digikey.com/product-detail/en/te-connectivity-alcoswitch-switches/TMS6T1B1M1QE/450-2109-ND/5125729" H 4200 1600 50  0001 C CNN
 F 4 "SWITCH TOGGLE SPST 3A 120V" H 4200 1600 50  0001 C CNN "Description"

Commit message: Updated footprint association
Parts:
- J6: footprint Connector:FanPinHeader_1x03_P2.54mm_Vertical -> Connector_PinHeader_2.54mm:PinHeader_1x03_P2.54mm_Vertical
- L2: footprint Aardonyx:L_Wuerth_WE_PDA_SMT-1280 -> Inductor_SMD:L_Wuerth_WE-PD-Typ-LS
Changed lines of the file:
@@
 EESchema Schematic File Version 4
-EELAYER 30 0
+LIBS:Aardonyx-cache
+EELAYER 29 0
 EELAYER END
 $Descr A4 11693 8268
@@
 F 0 "L2" V 6700 5050 50  0000 C CNN
 F 1 "3.3UH" V 6600 4900 50  0000 C CNN
-F 2 "Aardonyx:L_Wuerth_WE_PDA_SMT-1280" H 6650 4900 50  0001 C CNN
+F 2 "Inductor_SMD:L_Wuerth_WE-PD-Typ-LS" H 6650 4900 50  0001 C CNN
 F 3 "https://www.digikey.com/product-detail/en/w%C3%BCrth-elektronik/78477033/732-6781-2-ND/5168775" H 6650 4900 50  0001 C CNN
 F 4 "FIXED IND 3.3UH 6.6A 17 MOHM SMD" H 6650 4900 50  0001 C CNN "Description"
@@
 F 0 "J6" H 8750 4400 50  0000 L CNN
 F 1 "Conn_1x3_M" H 8650 4000 50  0000 L CNN
-F 2 "Connector:FanPinHeader_1x03_P2.54mm_Vertical" H 8750 4200 50  0001 C CNN
+F 2 "Connector_PinHeader_2.54mm:PinHeader_1x03_P2.54mm_Vertical" H 8750 4200 50  0001 C CNN
 F 3 "https://www.digikey.com/product-detail/en/amphenol-icc-fci/68000-203HLF/609-3464-ND/2023305" H 8750 4200 50  0001 C CNN
 F 4 "CONN HEADER VERT 3POS 2.54MM" H 8750 4200 50  0001 C CNN "Description"
