File: asic/e-class-aardonyx/board/Board_Design/sdram.sch (KiCad schematic (older format))
At the start: 13 parts, among them U2 IS42S32160F-TSOP2

Commit message: update
Parts:
- renumbered C27 to C45, C28 to C46, C29 to C47, C30 to C48, C31 to C49, C32 to C50, C33 to C51, C34 to C52, C35 to C53, C36 to C54, C37 to C55, C38 to C56, U2 to U4
Other:
- moved on the sheet: C45, C46, C47, C48, C49, C50, C51, C52, C53, C54, C55, C56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

Commit message: update
Parts:
- added C1, C2, C?: 0.1uf, symbol aardonyx:C_Small
- added J1: Conn_01x04, symbol Connector:Conn_01x04_Male
- added R100, R101, R? (x3): 10K, symbol aardonyx:R_US
- added R102: 0E, symbol aardonyx:R_US
- added U2: CDCE913PW, SOP65P640X120-14N, symbol aardonyx:CDCE913PW
- added Y1: 10MHz, symbol aardonyx:Crystal
Connections:
- net labels added: CLK
- wire segments 153 -> 211
Other:
- note added: "CLOCK MULTIPLIER\n"
- moved on the sheet: C45, C46, C47, C48, C49, C50, C51, C52, C53, C54, C55, C56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

Commit message: update
Parts:
- removed J1: Conn_01x04, symbol Connector:Conn_01x04_Male
- added J2: Conn_1x4, symbol aardonyx:Conn_01x04
- R19: renamed from R100; value 10K -> 4.7K
- R20: renamed from R101; value 10K -> 4.7K
- R21, R22, R23: renamed from R?; value 10K -> 4.7K
- Y2: renamed from Y1; value 10MHz -> 27MHz
- gave numbers to parts that had none: 1
- renumbered C45 to C18, C46 to C19, C47 to C20, C48 to C21, C49 to C22, C50 to C23, C51 to C24, C52 to C25, C53 to C26, C54 to C27, C55 to C28, C56 to C29, C1 to C31, C2 to C32, R102 to R24, U4 to U2, U2 to U3
Connections:
- net labels added: SDRAM_A0-12, SDRAM_D0-31, SDRAM_DQM0-3

Commit message: update
Parts:
- renumbered J2 to J4
Changed lines of the file:
@@
 encoding utf-8
 Sheet 3 7
-Title ""
+Title "AARDONYX_DEVELOPMENT_BOARD"
 Date ""
-Rev ""
-Comp ""
+Rev "R1V0"
+Comp "IIT_MADRAS"
 Comment1 ""
 Comment2 ""
@@
 SDRAM_CKE
 $Comp
-L aardonyx:V3P3 #PWR021
+L aardonyx:V3P3 #PWR024
 U 1 1 5DC441F1
 P 1650 1000
-F 0 "#PWR021" H 1800 950 50  0001 C CNN
+F 0 "#PWR024" H 1800 950 50  0001 C CNN
 F 1 "V3P3" H 1655 1175 50  0000 C CNN
 F 2 "" H 1650 1000 50  0001 C CNN
@@
 $EndComp
 $Comp
-L aardonyx:V3P3 #PWR022
+L aardonyx:V3P3 #PWR025
 U 1 1 5DC4BA51
 P 2550 2200
-F 0 "#PWR022" H 2700 2150 50  0001 C CNN
+F 0 "#PWR025" H 2700 2150 50  0001 C CNN
 F 1 "V3P3" H 2555 2375 50  0000 C CNN
 F 2 "" H 2550 2200 50  0001 C CNN
@@
 $EndComp
 $Comp
-L aardonyx:GND #PWR023
+L aardonyx:GND #PWR026
 U 1 1 5DC6067F
 P 3650 7450
-F 0 "#PWR023" H 3650 7200 50  0001 C CNN
+F 0 "#PWR026" H 3650 7200 50  0001 C CNN
 F 1 "GND" H 3655 7277 50  0000 C CNN
 F 2 "" H 3650 7450 50  0001 C CNN
@@
 $EndComp
 $Comp
-L aardonyx:GND #PWR024
+L aardonyx:GND #PWR027
 U 1 1 5DC61140
 P 4400 1800
-F 0 "#PWR024" H 4400 1550 50  0001 C CNN
+F 0 "#PWR027" H 4400 1550 50  0001 C CNN
 F 1 "GND" H 4405 1627 50  0000 C CNN
 F 2 "" H 4400 1800 50  0001 C CNN
@@
 P 7850 3050
 AR Path="/5D8B3740/5EFB4CF5" Ref="#PWR?"  Part="1"
-AR Path="/5D8B37B8/5EFB4CF5" Ref="#PWR030"  Part="1"
-F 0 "#PWR030" H 7850 2800 50  0001 C CNN
+AR Path="/5D8B37B8/5EFB4CF5" Ref="#PWR033"  Part="1"
+F 0 "#PWR033" H 7850 2800 50  0001 C CNN
 F 1 "GND" H 7855 2877 50  0000 C CNN
 F 2 "" H 7850 3050 50  0001 C CNN
@@
 P 9850 1800
 AR Path="/5D8B3740/5EFB4CFB" Ref="#PWR?"  Part="1"
-AR Path="/5D8B37B8/5EFB4CFB" Ref="#PWR031"  Part="1"
-F 0 "#PWR031" H 10000 1750 50  0001 C CNN
+AR Path="/5D8B37B8/5EFB4CFB" Ref="#PWR034"  Part="1"
+F 0 "#PWR034" H 10000 1750 50  0001 C CNN
 F 1 "V3P3" H 9855 1975 50  0000 C CNN
 F 2 "" H 9850 1800 50  0001 C CNN
@@
 P 7000 1850
 AR Path="/5D8B3740/5EFB4D20" Ref="#PWR?"  Part="1"
-AR Path="/5D8B37B8/5EFB4D20" Ref="#PWR027"  Part="1"
-F 0 "#PWR027" H 7150 1800 50  0001 C CNN
+AR Path="/5D8B37B8/5EFB4D20" Ref="#PWR030"  Part="1"
+F 0 "#PWR030" H 7150 1800 50  0001 C CNN
 F 1 "V3P3" H 7005 2025 50  0000 C CNN
 F 2 "" H 7000 1850 50  0001 C CNN
@@
 P 10150 2150
 AR Path="/5D8B3740/5EFB4D57" Ref="#PWR?"  Part="1"
-AR Path="/5D8B37B8/5EFB4D57" Ref="#PWR032"  Part="1"
-F 0 "#PWR032" H 10150 1900 50  0001 C CNN
+AR Path="/5D8B37B8/5EFB4D57" Ref="#PWR035"  Part="1"
+F 0 "#PWR035" H 10150 1900 50  0001 C CNN
 F 1 "GND" H 10155 1977 50  0000 C CNN
 F 2 "" H 10150 2150 50  0001 C CNN
@@
 P 6650 2300
 AR Path="/5D8B3740/5EFB4D70" Ref="#PWR?"  Part="1"
-AR Path="/5D8B37B8/5EFB4D70" Ref="#PWR025"  Part="1"
-F 0 "#PWR025" H 6800 2250 50  0001 C CNN
+AR Path="/5D8B37B8/5EFB4D70" Ref="#PWR028"  Part="1"
+F 0 "#PWR028" H 6800 2250 50  0001 C CNN
 F 1 "V3P3" H 6655 2475 50  0000 C CNN
 F 2 "" H 6650 2300 50  0001 C CNN
@@
 P 6750 2750
 AR Path="/5D8B3740/5EFB4D78" Ref="#PWR?"  Part="1"
-AR Path="/5D8B37B8/5EFB4D78" Ref="#PWR026"  Part="1"
-F 0 "#PWR026" H 6750 2500 50  0001 C CNN
+AR Path="/5D8B37B8/5EFB4D78" Ref="#PWR029"  Part="1"
+F 0 "#PWR029" H 6750 2500 50  0001 C CNN
 F 1 "GND" H 6755 2577 50  0000 C CNN
 F 2 "" H 6750 2750 50  0001 C CNN
@@
 P 7450 1700
 AR Path="/5D8B3740/5F91E22E" Ref="#PWR?"  Part="1"
-AR Path="/5D8B37B8/5F91E22E" Ref="#PWR028"  Part="1"
-F 0 "#PWR028" H 7450 1450 50  0001 C CNN
+AR Path="/5D8B37B8/5F91E22E" Ref="#PWR031"  Part="1"
+F 0 "#PWR031" H 7450 1450 50  0001 C CNN
 F 1 "GND" H 7455 1527 50  0000 C CNN
 F 2 "" H 7450 1700 50  0001 C CNN
@@
 P 7650 1350
 AR Path="/5D8B3740/5EFB4D62" Ref="#PWR?"  Part="1"
-AR Path="/5D8B37B8/5EFB4D62" Ref="#PWR029"  Part="1"
-F 0 "#PWR029" H 7800 1300 50  0001 C CNN
+AR Path="/5D8B37B8/5EFB4D62" Ref="#PWR032"  Part="1"
+F 0 "#PWR032" H 7800 1300 50  0001 C CNN
 F 1 "V3P3" H 7655 1525 50  0000 C CNN
 F 2 "" H 7650 1350 50  0001 C CNN
@@
 SDRAM_BA0
 $Comp
-L aardonyx:Conn_01x04 J2
+L aardonyx:Conn_01x04 J4
 U 1 1 63AEA5D7
 P 6350 2450
-F 0 "J2" H 6430 2442 50  0000 L CNN
+F 0 "J4" H 6430 2442 50  0000 L CNN
 F 1 "Conn_1x4" H 6200 2100 50  0000 L CNN
 F 2 "" H 6350 2450 50  0001 C CNN

Commit message: updare
Parts:
- added TP3, TP4: TestPoint, symbol aardonyx:TestPoint
- R22, R23: Field4 (none) -> NA
- R24: value 0E -> 22E
Connections:
- net at U3.8 (Y3): now also TP4.1
- net at U3.9 (Y2): now also TP3.1
Changed lines of the file:
@@
 AR Path="/5D8B37B8/5EFB4D80" Ref="R24"  Part="1"
 F 0 "R24" V 9900 2450 50  0000 C CNN
-F 1 "0E" V 9900 2750 50  0000 C CNN
+F 1 "22E" V 9900 2750 50  0000 C CNN
 F 2 "" V 9990 2590 50  0001 C CNN
 F 3 "~" H 9950 2600 50  0001 C CNN
@@
 AR Path="/5D8B3740/5F82D0FE" Ref="R?"  Part="1"
 AR Path="/5D8B37B8/5F82D0FE" Ref="R23"  Part="1"
-F 0 "R23" H 7500 2800 50  0000 L CNN
-F 1 "4.7K" H 7700 2800 50  0000 L CNN
+F 0 "R23" H 7450 2800 50  0000 L CNN
+F 1 "4.7K" H 7650 2700 50  0000 L CNN
 F 2 "" V 7690 2790 50  0001 C CNN
 F 3 "~" H 7650 2800 50  0001 C CNN
+F 4 "NA" H 7750 2800 50  0000 C CNN "Field4"
 	1    7650 2800
 	1    0    0    -1
@@
 F 2 "" V 7690 1990 50  0001 C CNN
 F 3 "~" H 7650 2000 50  0001 C CNN
+F 4 "NA" H 7750 2050 50  0000 C CNN "Field4"
 	1    7650 2000
 	1    0    0    -1
@@
 	-1   0    0    -1
 $EndComp
+$Comp
+L aardonyx:TestPoint TP3
+U 1 1 5E889222
+P 9600 2700
+F 0 "TP3" V 9600 2888 50  0000 L CNN
+F 1 "TestPoint" V 9645 2888 50  0001 L CNN
+F 2 "" H 9800 2700 50  0001 C CNN
+F 3 "~" H 9800 2700 50  0001 C CNN
+	1    9600 2700
+	0    1    1    0
+$EndComp
+$Comp
+L aardonyx:TestPoint TP4
+U 1 1 5E88A45B
+P 9600 2800
+F 0 "TP4" V 9600 2988 50  0000 L CNN
+F 1 "TestPoint" V 9645 2988 50  0001 L CNN
+F 2 "" H 9800 2800 50  0001 C CNN
+F 3 "~" H 9800 2800 50  0001 C CNN
+	1    9600 2800
+	0    1    1    0
+$EndComp
+Wire Wire Line
+	9550 2700 9600 2700
+Wire Wire Line
+	9600 2800 9550 2800
 Wire Bus Line
 	1550 5700 1550 6100
