File: asic/e-class-aardonyx/board/Board_Design/sdram.sch (KiCad schematic (older format))
At the start: 30 parts, among them J4 Conn_1x4, U15 SKT32E, U2 IS42S32160F-TSOP2, U3 CDCE913PW, Y2 27MHz

Commit message: Update Footprint
Parts:
- J4: footprint (none) -> Connector_PinHeader_2.54mm:PinHeader_1x04_P2.54mm_Vertical
- U2: footprint (none) -> Aardonyx:TSSOP-II-86_10.16x22.2mm_P0.5mm
Changed lines of the file:
@@
 EESchema Schematic File Version 4
-LIBS:Aardonyx-cache
-EELAYER 29 0
+EELAYER 30 0
 EELAYER END
 $Descr A4 11693 8268
@@
 F 0 "U2" H 2350 6950 50  0000 C CNN
 F 1 "IS42S32160F-TSOP2" H 3050 4800 50  0000 C CNN
-F 2 "" H 3100 4950 50  0001 C CNN
+F 2 "Aardonyx:TSSOP-II-86_10.16x22.2mm_P0.5mm" H 3100 4950 50  0001 C CNN
 F 3 "https://www.digikey.in/product-detail/en/issi-integrated-silicon-solution-inc/IS42S32160F-7TLI/706-1417-5-ND/5319838" H 3100 4950 50  0001 C CNN
 F 4 "IC DRAM 512M PARALLEL 86TSOP II" H 3100 4800 50  0001 C CNN "Description"
@@
 F 0 "J4" H 6430 2442 50  0000 L CNN
 F 1 "Conn_1x4" H 6200 2100 50  0000 L CNN
-F 2 "" H 6350 2450 50  0001 C CNN
+F 2 "Connector_PinHeader_2.54mm:PinHeader_1x04_P2.54mm_Vertical" H 6350 2450 50  0001 C CNN
 F 3 "https://www.digikey.com/product-detail/en/amphenol-icc-fci/68000-404HLF/609-3262-ND/1878463" H 6350 2450 50  0001 C CNN
 F 4 "CONN HEADER VERT 4POS 2.54MM" H 6350 2450 50  0001 C CNN "Description"
@@
 Text Notes 7200 4950 0    200  ~ 40
 SKT32E NC PINS\n
+Text Notes 4250 6950 0    50   ~ 0
+512Mb - SDRAM (16 x 32Mbit)
+Text Notes 4250 7100 0    50   ~ 0
+86-pin TSOP-ll
 Wire Bus Line
 	1550 5700 1550 6100
@@
 Wire Bus Line
 	4650 3000 4650 6600
-Text Notes 4250 6950 0    50   ~ 0
-512Mb - SDRAM (16 x 32Mbit)
-Text Notes 4250 7100 0    50   ~ 0
-86-pin TSOP-ll
 $EndSCHEMATC

Commit message: update foot print & componenet placement
Parts:
- Y2: footprint Crystal:Crystal_SMD_HC49-SD_HandSoldering -> Aardonyx:Crystal_SMD_ROHS_CSM_7XDN_HandSoldering
Changed lines of the file:
@@
 F 0 "Y2" H 8750 1200 50  0000 L CNN
 F 1 "27MHz" H 8650 1500 50  0000 L CNN
-F 2 "Crystal:Crystal_SMD_HC49-SD_HandSoldering" H 8750 1350 50  0001 C CNN
+F 2 "Aardonyx:Crystal_SMD_ROHS_CSM_7XDN_HandSoldering" H 8750 1350 50  0001 C CNN
 F 3 "https://www.digikey.in/product-detail/en/ecs-inc/ECS-270-18-5PX-F-TR/XC1002CT-ND/813243" H 8750 1350 50  0001 C CNN
 F 4 "CRYSTAL 27.0000MHZ 18PF SMD" H 8750 1350 50  0001 C CNN "Description"
