File: asic/e-class-aardonyx/board/Board_Design/soc.sch (KiCad schematic (older format))
At the start: 106 parts, among them SW3 SW_DIP_x03, U15 SKT32E

Commit message: update bom
Parts:
- R131, R132: Description (none) -> RES SMD 0 OHM JUMPER 1/8W 0805; Digikey PartNumber (none) -> 541-0.0ACT-ND; Manufactured Part Number (none) -> CRCW08050000Z0EA; Maufaturer (none) -> Vishay Dale

Commit message: update BOM
Parts:
- C63, C64, C65, C66, C67, C68, C69, C70, C71, C72, C73, C74, C75, C76, C77, C78, C79, C80, C81, C82, C83, C84, C85, C86, C87, C88, C89, C90: Description CAP CER 0.1UF 16V X7R 0402 -> CAP CER 0.1UF 25V X7R 0402; Digikey PartNumber 490-6328-1-ND -> 478-10050-1-ND; Manufactured Part Number GRM155R71C104KA88J -> 04023C104JAT2A; Maufaturer Murata -> AVX Corporation
- R100, R101, R102, R103, R104, R105, R106, R107, R108, R109, R110, R111, R112, R113, R114, R115, R116, R117, R118, R119, R120, R121, R122, R123, R124, R125, R126, R127, R57, R58, R59, R60, R61, R62, R63, R64, R65, R66, R67, R68, R69, R70, R71, R72, R73, R74, R75, R76, R77, R78, R79, R80, R81, R82, R83, R84, R85, R86, R87, R88, R89, R90, R91, R92, R93, R94, R95, R96, R97, R98, R99: Description (none) -> RES SMD 22 OHM 1% 1/16W 0402; Digikey PartNumber (none) -> 311-22.0LRCT-ND; Manufactured Part Number (none) -> RC0402FR-0722RL; Maufaturer (none) -> Yageo
- R131, R132: Description RES SMD 0 OHM JUMPER 1/8W 0805 -> RES SMD 0 OHM JUMPER 1/16W 0402; Digikey PartNumber 541-0.0ACT-ND -> 541-0.0JCT-ND; Manufactured Part Number CRCW08050000Z0EA -> CRCW04020000Z0ED

Commit message: updated BOM
Parts:
- C63, C64, C65, C66, C67, C68, C69, C70, C71, C72, C73, C74, C75, C76, C77, C78, C79, C80, C81, C82, C83, C84, C85, C86, C87, C88, C89, C90: value 0.1uF -> 0.1UF,0402
- R100, R101, R102, R103, R104, R105, R106, R107, R108, R109, R110, R111, R112, R113, R114, R115, R116, R117, R118, R119, R120, R121, R122, R123, R124, R125, R126, R127, R57, R58, R59, R60, R61, R62, R63, R64, R65, R66, R67, R68, R69, R70, R71, R72, R73, R74, R75, R76, R77, R78, R79, R80, R81, R82, R83, R84, R85, R86, R87, R88, R89, R90, R91, R92, R93, R94, R95, R96, R97, R98, R99: value 22E -> 22E,0402
- R128, R129, R130: value 10K -> 10KE,0805
- R131, R132: value 0E -> 0E, 0402
- SW3: Description (none) -> SWITCH SLIDE DIP SPST 25MA 24V; Digikey PartNumber (none) -> 732-3833-5-ND; Field4 (none) -> 732-3833-5-ND; Manufactured Part Number (none) -> 418117270903; Maufaturer (none) -> Würth Elektronik
- U15: Description (none) -> Aardonyx 32bit EClass ASIC; Digikey PartNumber (none) -> CUSTOM MADE; Manufactured Part Number (none) -> SKT32E; Maufaturer (none) -> SCL

Commit message: updated commented pending schematic
Parts:
- removed U15: SKT32E, symbol Aardonyx-rescue:SKT32E-aardonyx
- added U15: SKT32E, symbol Aardonyx-rescue:SKT32E-skt32e_asic
Connections:
- net labels added: IO_[0..7], IO_[8..13], SDRAM_A[0..12], SDRAM_DQM[0..3], SDRAM_D[0..31]
- net labels removed: IO_0-7, IO_8-13, SDRAM_A0-12, SDRAM_D0-31, SDRAM_DQM0-3
Other:
- moved on the sheet: R128, R129, R130, R131, R132, R57, R58, R59, R60, R61, R62, R63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

Commit message: updated footprint for netlist
Parts:
- C63, C64, C65, C66, C67, C68, C69, C70, C71, C72, C73, C74, C75, C76, C77, C78, C79, C80, C81, C82, C83, C84, C85, C86, C87, C88, C89, C90: footprint (none) -> Capacitor_SMD:C_0402_1005Metric
- R100, R101, R102, R103, R104, R105, R106, R107, R108, R109, R110, R111, R112, R113, R114, R115, R116, R117, R118, R119, R120, R121, R122, R123, R124, R125, R126, R127, R131, R132, R57, R58, R59, R60, R61, R62, R63, R64, R65, R66, R67, R68, R69, R70, R71, R72, R73, R74, R75, R76, R77, R78, R79, R80, R81, R82, R83, R84, R85, R86, R87, R88, R89, R90, R91, R92, R93, R94, R95, R96, R97, R98, R99: footprint (none) -> Resistor_SMD:R_0402_1005Metric
- R128, R129, R130: footprint (none) -> Resistor_SMD:R_0805_2012Metric
- U15: footprint (none) -> Aardonyx:SKT32E_IITM

Commit message: updated footprint
Parts:
- SW3: footprint (none) -> Button_Switch_THT:SW_DIP_SPSTx03_Slide_6.7x9.18mm_W7.62mm_P2.54mm_LowProfile
Changed lines of the file:
@@
 F 0 "SW3" H 9850 5950 50  0000 C CNN
 F 1 "SW_DIP_x03" H 10100 5450 50  0000 C CNN
-F 2 "" H 9900 5600 50  0001 C CNN
+F 2 "Button_Switch_THT:SW_DIP_SPSTx03_Slide_6.7x9.18mm_W7.62mm_P2.54mm_LowProfile" H 9900 5600 50  0001 C CNN
 F 3 "https://www.digikey.com/product-detail/en/w%C3%BCrth-elektronik/418117270903/732-3833-5-ND/3174487" H 9900 5600 50  0001 C CNN
 F 4 "	SWITCH SLIDE DIP SPST 25MA 24V" H 9900 5600 50  0001 C CNN "Description"

Commit message: Updated schematic
Parts:
- removed C85: 0.1UF,0402, Capacitor_SMD:C_0402_1005Metric, symbol Aardonyx-rescue:C_Small-aardonyx
- added D6, D7, D8: LED,1206, LED_SMD:LED_0603_1608Metric, symbol Device:LED_ALT
- added R42, R43, R44: 220E,0402, Resistor_SMD:R_0402_1005Metric, symbol Aardonyx-rescue:R_US-aardonyx
- U15: Description (none) -> E class Shakti Processor; Digikey PartNumber (none) -> NA; Manufactured Part Number (none) -> SKT32E; Maufaturer (none) -> SCL / IITM
Connections:
- net GNDREF: now also D6.1 (K), D7.1 (K), D8.1 (K)
- net IO_13: now also R42.1
- net IO_14: now also R43.1
- net IO_15: now also R44.1
- new net: D6.2 (A), R42.2
- new net: D7.2 (A), R43.2
- new net: D8.2 (A), R44.2
Other:
- note added: "DEBUG LEDS\n"
- moved on the sheet: R128, R129, R130, R131, R132, SW3
