File: asic/e-class-aardonyx/board/Board_Design/soc.sch (KiCad schematic (older format))
At the start: 111 parts, among them SW3 SW_DIP_x03, U15 SKT32E

Commit message: add bom
Parts:
- D6, D7, D8: Maufaturer Lumex Opto/Components Inc. -> Lumex Opto/Components Inc.
- SW3: Description SWITCH SLIDE DIP SPST 25MA 24V -> SWITCH SLIDE DIP SPST 25MA 24V; Digikey PartNumber 732-3833-5-ND -> 732-3833-5-ND
Changed lines of the file:
@@
 F 2 "Button_Switch_THT:SW_DIP_SPSTx03_Slide_6.7x9.18mm_W7.62mm_P2.54mm_LowProfile" H 9950 5700 50  0001 C CNN
 F 3 "https://www.digikey.com/product-detail/en/w%C3%BCrth-elektronik/418117270903/732-3833-5-ND/3174487" H 9950 5700 50  0001 C CNN
-F 4 "	SWITCH SLIDE DIP SPST 25MA 24V" H 9950 5700 50  0001 C CNN "Description"
-F 5 "	732-3833-5-ND" H 9950 5700 50  0001 C CNN "Digikey PartNumber"
+F 4 "SWITCH SLIDE DIP SPST 25MA 24V" H 9950 5700 50  0001 C CNN "Description"
+F 5 "732-3833-5-ND" H 9950 5700 50  0001 C CNN "Digikey PartNumber"
 F 6 "732-3833-5-ND" H 9950 5700 50  0001 C CNN "Field4"
 F 7 "418117270903" H 9950 5700 50  0001 C CNN "Manufactured Part Number"
@@
 F 5 "67-1002-1-ND" H 7850 5200 50  0001 C CNN "Digikey PartNumber"
 F 6 "SML-LX1206GW-TR" H 7850 5200 50  0001 C CNN "Manufactured Part Number"
-F 7 "	Lumex Opto/Components Inc." H 7850 5200 50  0001 C CNN "Maufaturer"
+F 7 "Lumex Opto/Components Inc." H 7850 5200 50  0001 C CNN "Maufaturer"
 	1    7850 5200
 	-1   0    0    1
@@
 F 5 "67-1002-1-ND" H 7850 5450 50  0001 C CNN "Digikey PartNumber"
 F 6 "SML-LX1206GW-TR" H 7850 5450 50  0001 C CNN "Manufactured Part Number"
-F 7 "	Lumex Opto/Components Inc." H 7850 5450 50  0001 C CNN "Maufaturer"
+F 7 "Lumex Opto/Components Inc." H 7850 5450 50  0001 C CNN "Maufaturer"
 	1    7850 5450
 	-1   0    0    1
@@
 F 5 "67-1002-1-ND" H 7850 5800 50  0001 C CNN "Digikey PartNumber"
 F 6 "SML-LX1206GW-TR" H 7850 5800 50  0001 C CNN "Manufactured Part Number"
-F 7 "	Lumex Opto/Components Inc." H 7850 5800 50  0001 C CNN "Maufaturer"
+F 7 "Lumex Opto/Components Inc." H 7850 5800 50  0001 C CNN "Maufaturer"
 	1    7850 5800
 	-1   0    0    1

Commit message: Updated few components
Parts:
- R42, R43, R44: Description RES SMD 120 OHM 1% 1/16W 0402 -> RES SMD 220 OHM 1% 1/16W 0402; Digikey PartNumber 311-120LRCT-ND -> 311-220LRDKR-ND; Manufactured Part Number RC0402FR-07120RL -> RC0402FR-07220RL
Changed lines of the file:
@@
 EESchema Schematic File Version 4
-EELAYER 30 0
+LIBS:Aardonyx-cache
+EELAYER 29 0
 EELAYER END
 $Descr A4 11693 8268
@@
 F 1 "220E,0402" V 7300 4950 50  0000 L CNN
 F 2 "Resistor_SMD:R_0402_1005Metric" V 7440 5190 50  0001 C CNN
-F 3 "https://www.digikey.in/product-detail/en/yageo/RC1206JR-07120RL/311-120ERCT-ND/732162" H 7400 5200 50  0001 C CNN
-F 4 "RES SMD 120 OHM 1% 1/16W 0402" H 7400 5200 50  0001 C CNN "Description"
-F 5 "311-120LRCT-ND" H 7400 5200 50  0001 C CNN "Digikey PartNumber"
-F 6 "RC0402FR-07120RL" H 7400 5200 50  0001 C CNN "Manufactured Part Number"
+F 3 "https://www.digikey.in/product-detail/en/yageo/RC0402FR-07220RL/311-220LRDKR-ND/732459" H 7400 5200 50  0001 C CNN
+F 4 "RES SMD 220 OHM 1% 1/16W 0402" H 7400 5200 50  0001 C CNN "Description"
+F 5 "311-220LRDKR-ND" H 7400 5200 50  0001 C CNN "Digikey PartNumber"
+F 6 "RC0402FR-07220RL" H 7400 5200 50  0001 C CNN "Manufactured Part Number"
 F 7 "Yageo" H 7400 5200 50  0001 C CNN "Maufaturer"
 	1    7400 5200
@@
 F 1 "220E,0402" V 7300 5200 50  0000 L CNN
 F 2 "Resistor_SMD:R_0402_1005Metric" V 7440 5440 50  0001 C CNN
-F 3 "https://www.digikey.in/product-detail/en/yageo/RC1206JR-07120RL/311-120ERCT-ND/732162" H 7400 5450 50  0001 C CNN
-F 4 "RES SMD 120 OHM 1% 1/16W 0402" H 7400 5450 50  0001 C CNN "Description"
-F 5 "311-120LRCT-ND" H 7400 5450 50  0001 C CNN "Digikey PartNumber"
-F 6 "RC0402FR-07120RL" H 7400 5450 50  0001 C CNN "Manufactured Part Number"
+F 3 "https://www.digikey.in/product-detail/en/yageo/RC0402FR-07220RL/311-220LRDKR-ND/732459" H 7400 5450 50  0001 C CNN
+F 4 "RES SMD 220 OHM 1% 1/16W 0402" H 7400 5450 50  0001 C CNN "Description"
+F 5 "311-220LRDKR-ND" H 7400 5450 50  0001 C CNN "Digikey PartNumber"
+F 6 "RC0402FR-07220RL" H 7400 5450 50  0001 C CNN "Manufactured Part Number"
 F 7 "Yageo" H 7400 5450 50  0001 C CNN "Maufaturer"
 	1    7400 5450
@@
 F 1 "220E,0402" V 7300 5550 50  0000 L CNN
 F 2 "Resistor_SMD:R_0402_1005Metric" V 7440 5790 50  0001 C CNN
-F 3 "https://www.digikey.in/product-detail/en/yageo/RC1206JR-07120RL/311-120ERCT-ND/732162" H 7400 5800 50  0001 C CNN
-F 4 "RES SMD 120 OHM 1% 1/16W 0402" H 7400 5800 50  0001 C CNN "Description"
-F 5 "311-120LRCT-ND" H 7400 5800 50  0001 C CNN "Digikey PartNumber"
-F 6 "RC0402FR-07120RL" H 7400 5800 50  0001 C CNN "Manufactured Part Number"
+F 3 "https://www.digikey.in/product-detail/en/yageo/RC0402FR-07220RL/311-220LRDKR-ND/732459" H 7400 5800 50  0001 C CNN
+F 4 "RES SMD 220 OHM 1% 1/16W 0402" H 7400 5800 50  0001 C CNN "Description"
+F 5 "311-220LRDKR-ND" H 7400 5800 50  0001 C CNN "Digikey PartNumber"
+F 6 "RC0402FR-07220RL" H 7400 5800 50  0001 C CNN "Manufactured Part Number"
 F 7 "Yageo" H 7400 5800 50  0001 C CNN "Maufaturer"
 	1    7400 5800

Commit message: updated component
Connections:
- net I2C0_SCL: no longer U15.37 (I2C0_SDA)
- new net I2C0_SDA: U15.37 (I2C0_SDA)
Changed lines of the file:
@@
 QSPI0_IO3
 Text HLabel 4900 2250 2    50   BiDi ~ 0
+I2C0_SDA
+Text HLabel 4900 2350 2    50   BiDi ~ 0
 I2C0_SCL
-Text HLabel 4900 2350 2    50   BiDi ~ 0
-I2C0_SDA
 Text HLabel 4900 1350 2    50   Output ~ 0
 UART0_TX

Commit message: Added few components
Parts:
- R128, R129, R130: value 10KE,0805 -> 10KE,0402; footprint Resistor_SMD:R_0805_2012Metric -> Resistor_SMD:R_0402_1005Metric; Description RES SMD 10K OHM 1% 1/8W 0805 -> RES 10K OHM 5% 1/8W 0402; Digikey PartNumber 311-10.0KCRCT-ND -> 2019-SG73S1ETTP103JCT-ND; Manufactured Part Number RC0805FR-0710KL -> SG73S1ETTP103J; Maufaturer Yageo -> KOA Speer Electronics, Inc.
Connections:
- net BOOT_MODE0: now also R128.1, SW3.3; no longer R130.1, SW3.1
- net TEST_MODE: now also R130.1, SW3.1; no longer R128.1, SW3.3
Changed lines of the file:
@@
 	10900 5500 10900 5350
 Text Label 8850 5700 0    39   ~ 0
-TEST_MODE
+BOOT_MODE0
 Text Label 8850 5600 0    39   ~ 0
 BOOT_MODE1
 Text Label 8850 5500 0    39   ~ 0
-BOOT_MODE0
+TEST_MODE
 $Comp
 L Aardonyx-rescue:R_US-aardonyx R131
@@
 P 9600 5900
 F 0 "R130" V 9550 6000 50  0000 C CNN
-F 1 "10KE,0805" V 9650 5650 50  0000 C CNN
-F 2 "Resistor_SMD:R_0805_2012Metric" V 9640 5890 50  0001 C CNN
-F 3 "https://www.digikey.in/product-detail/en/yageo/RC0805FR-0710KL/311-10-0KCRCT-ND/730482" H 9600 5900 50  0001 C CNN
-F 4 "RES SMD 10K OHM 1% 1/8W 0805" H 9600 5900 50  0001 C CNN "Description"
-F 5 "311-10.0KCRCT-ND" H 9600 5900 50  0001 C CNN "Digikey PartNumber"
-F 6 "RC0805FR-0710KL" H 9600 5900 50  0001 C CNN "Manufactured Part Number"
-F 7 "Yageo" H 9600 5900 50  0001 C CNN "Maufaturer"
+F 1 "10KE,0402" V 9650 5650 50  0000 C CNN
+F 2 "Resistor_SMD:R_0402_1005Metric" V 9640 5890 50  0001 C CNN
+F 3 "https://www.digikey.in/product-detail/en/koa-speer-electronics-inc/SG73S1ETTP103J/2019-SG73S1ETTP103JCT-ND/10280218" H 9600 5900 50  0001 C CNN
+F 4 "RES 10K OHM 5% 1/8W 0402" H 9600 5900 50  0001 C CNN "Description"
+F 5 "2019-SG73S1ETTP103JCT-ND" H 9600 5900 50  0001 C CNN "Digikey PartNumber"
+F 6 "SG73S1ETTP103J" H 9600 5900 50  0001 C CNN "Manufactured Part Number"
+F 7 "KOA Speer Electronics, Inc." H 9600 5900 50  0001 C CNN "Maufaturer"
 	1    9600 5900
 	1    0    0    -1
@@
 P 9400 5900
 F 0 "R129" V 9350 6050 50  0000 C CNN
-F 1 "10KE,0805" V 9450 5750 50  0000 C CNN
-F 2 "Resistor_SMD:R_0805_2012Metric" V 9440 5890 50  0001 C CNN
-F 3 "https://www.digikey.in/product-detail/en/yageo/RC0805FR-0710KL/311-10-0KCRCT-ND/730482" H 9400 5900 50  0001 C CNN
-F 4 "RES SMD 10K OHM 1% 1/8W 0805" H 9400 5900 50  0001 C CNN "Description"
-F 5 "311-10.0KCRCT-ND" H 9400 5900 50  0001 C CNN "Digikey PartNumber"
-F 6 "RC0805FR-0710KL" H 9400 5900 50  0001 C CNN "Manufactured Part Number"
-F 7 "Yageo" H 9400 5900 50  0001 C CNN "Maufaturer"
+F 1 "10KE,0402" V 9450 5750 50  0000 C CNN
+F 2 "Resistor_SMD:R_0402_1005Metric" V 9440 5890 50  0001 C CNN
+F 3 "https://www.digikey.in/product-detail/en/koa-speer-electronics-inc/SG73S1ETTP103J/2019-SG73S1ETTP103JCT-ND/10280218" H 9400 5900 50  0001 C CNN
+F 4 "RES 10K OHM 5% 1/8W 0402" H 9400 5900 50  0001 C CNN "Description"
+F 5 "2019-SG73S1ETTP103JCT-ND" H 9400 5900 50  0001 C CNN "Digikey PartNumber"
+F 6 "SG73S1ETTP103J" H 9400 5900 50  0001 C CNN "Manufactured Part Number"
+F 7 "KOA Speer Electronics, Inc." H 9400 5900 50  0001 C CNN "Maufaturer"
 	1    9400 5900
 	1    0    0    -1
@@
 P 9250 5900
 F 0 "R128" V 9150 6000 50  0000 C CNN
-F 1 "10KE,0805" V 9200 5600 50  0000 C CNN
-F 2 "Resistor_SMD:R_0805_2012Metric" V 9290 5890 50  0001 C CNN
-F 3 "https://www.digikey.in/product-detail/en/yageo/RC0805FR-0710KL/311-10-0KCRCT-ND/730482" H 9250 5900 50  0001 C CNN
-F 4 "RES SMD 10K OHM 1% 1/8W 0805" H 9250 5900 50  0001 C CNN "Description"
-F 5 "311-10.0KCRCT-ND" H 9250 5900 50  0001 C CNN "Digikey PartNumber"
-F 6 "RC0805FR-0710KL" H 9250 5900 50  0001 C CNN "Manufactured Part Number"
-F 7 "Yageo" H 9250 5900 50  0001 C CNN "Maufaturer"
+F 1 "10KE,0402" V 9200 5600 50  0000 C CNN
+F 2 "Resistor_SMD:R_0402_1005Metric" V 9290 5890 50  0001 C CNN
+F 3 "https://www.digikey.in/product-detail/en/koa-speer-electronics-inc/SG73S1ETTP103J/2019-SG73S1ETTP103JCT-ND/10280218" H 9250 5900 50  0001 C CNN
+F 4 "RES 10K OHM 5% 1/8W 0402" H 9250 5900 50  0001 C CNN "Description"
+F 5 "2019-SG73S1ETTP103JCT-ND" H 9250 5900 50  0001 C CNN "Digikey PartNumber"
+F 6 "SG73S1ETTP103J" H 9250 5900 50  0001 C CNN "Manufactured Part Number"
+F 7 "KOA Speer Electronics, Inc." H 9250 5900 50  0001 C CNN "Maufaturer"
 	1    9250 5900
 	1    0    0    -1
