File: asic/e-class-aardonyx/board/Board_Design/arduino_header.sch (KiCad schematic (older format))
At the start: 22 parts, among them U10 CAT24M01WI-GT3, U4 IS25LP256x-xM, U5 LSF0108PWR, U6 LSF0108PWR

Commit message: update
Parts:
- gave numbers to parts that had none: 5
- renumbered C39 to C57, C40 to C58, C41 to C59, C42 to C60, C43 to C61, C44 to C62, R4 to R63, R5 to R64, R6 to R65, R7 to R66, R8 to R67, R9 to R68, R10 to R69, U10 to U5, U4 to U6, U5 to U7, U6 to U8

Commit message: update
Parts:
- added C82, C83: 0.1UF, symbol aardonyx:C_Small
- added R103: 10K, symbol aardonyx:R_US
- added U13: MCP3008, symbol aardonyx:MCP3008
- renumbered J3 to J4, J4 to J5, J5 to J6, J6 to J7, J7 to J8, R63 to R78, R64 to R79, R65 to R80, R66 to R81, R67 to R82, R68 to R83, R69 to R84
Connections:
- net labels added: SPI0_CLK, SPI0_MISO, SPI0_MOSI, SPI0_nCS
- wire segments 158 -> 186
- no-connect marks 1 -> 3
Other:
- moved on the sheet: C59, C62, J4, J5, J6, J7, J8, R84, U8

Commit message: update
Parts:
- added J10, J11, J12, J13, J5, J6, J7, J9: Conn_1x3_M, symbol aardonyx:Conn_1x3_M
- added J14: Conn_1x8, symbol aardonyx:Conn_1x8
- added J15, J16: Conn_1x6_F, symbol aardonyx:Conn_1x6_F
- added J8: Conn_1X4, symbol aardonyx:Conn_01x04
- renumbered C57 to C47, C58 to C48, C82 to C49, C83 to C50, C60 to C51, C61 to C52, C59 to C53, C62 to C54, J6 to J17, J4 to J18, J5 to J19, J7 to J20, J8 to J21, R78 to R30, R79 to R31, R80 to R32, R81 to R33, R82 to R34, R103 to R35, R83 to R36, R84 to R37, U13 to U7, U7 to U8, U8 to U9
Connections:
- net labels added: A7, A8, I2C0_SCL_E, I2C0_SCL_H, I2C0_SDA_E, I2C0_SDA_H, IO_0-7, IO_14, IO_15, IO_8-13, QSPI0_CLK_F, QSPI0_CLK_H, QSPI0_IO0_F, QSPI0_IO0_H, QSPI0_IO1_F, QSPI0_IO1_H, QSPI0_IO2_F, QSPI0_IO2_H, QSPI0_IO3_F, QSPI0_IO3_H, QSPI0_NCS_F, QSPI0_NCS_H, RESET_AH, SPI1_CLK, SPI1_MISO, SPI1_MOSI, SPI1_nCS
- wire segments 186 -> 248
- no-connect marks 3 -> 1
Other:
- note added: "ADC\n"
- note added: "ARDUINO HEADER\n"
- moved on the sheet: C47, C48, C49, C50, C51, C52, C53, C54, J17, J18, J19, J20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

Commit message: update
Parts:
- renumbered J8 to J10, J9 to J11, J10 to J12, J11 to J13, J12 to J14, J13 to J15, J14 to J16, J15 to J17, J16 to J18, J17 to J19, J18 to J20, J19 to J21, J20 to J22, J21 to J23, J5 to J7, J6 to J8, J7 to J9

Commit message: updare
Parts:
- removed J11, J12, J13, J14, J15, J7, J8: Conn_1x3_M, symbol aardonyx:Conn_1x3_M
- renumbered J17 to J10, J18 to J11, J19 to J12, J20 to J13, J21 to J14, J22 to J15, J23 to J16, J10 to J7, J9 to J8, J16 to J9
Connections:
- net I2C0_SCL_E is gone; now on net I2C0_SCL: R34.2, U5.6 (SCL)
- net I2C0_SCL_H is gone; now on net I2C0_SCL: J7.2 (Pin_2)
- net I2C0_SDA_E is gone; now on net I2C0_SDA: R33.2, U5.5 (SDA)
- net I2C0_SDA_H is gone; now on net I2C0_SDA: J7.3 (Pin_3)
- net QSPI0_CLK_F is gone; now on net QSPI0_CLK: U6.16 (SCK)
- net QSPI0_CLK_H is gone; now on net QSPI0_CLK: J9.3 (Pin_3)
- net QSPI0_IO0_F is gone; now on net QSPI0_IO0: U6.15 (SI/IO0)
- net QSPI0_IO0_H is gone; now on net QSPI0_IO0: J9.4 (Pin_4)
- net QSPI0_IO1_F is gone; now on net QSPI0_IO1: U6.8 (SO/IO1)
- net QSPI0_IO1_H is gone; now on net QSPI0_IO1: J9.5 (Pin_5)
- net QSPI0_IO2_F is gone; now on net QSPI0_IO2: R31.2, U6.9 (~WP~/IO2)
- net QSPI0_IO2_H is gone; now on net QSPI0_IO2: J9.6 (Pin_6)
- net QSPI0_IO3_F is gone; now on net QSPI0_IO3: R30.2, U6.1 (~HOLD~/IO3)
- net QSPI0_IO3_H is gone; now on net QSPI0_IO3: J9.7 (Pin_7)
Other:
- moved on the sheet: C47, C48, J7, J8, J9, R30, R31, R32, R33, R34, U5, U6

Commit message: update
Parts:
- removed U7: MCP3008, symbol aardonyx:MCP3008
- added U?: ADC108S102CIMTX, symbol aardonyx:ADC108S102CIMTX_NOPB
Connections:
- net A0: now also U?.4 (IN0)
- net A1: now also U?.5 (IN1)
- net A2: now also U?.6 (IN2)
- net A3: now also U?.7 (IN3)
- net A4: now also U?.8 (IN4)
- net A5: now also U?.9 (IN5)
- net A7: now also U?.10 (IN6)
- net A8: now also U?.11 (IN7)
- net GNDREF: now also U?.12 (DGND), U?.3 (AGND)
- net SPI0_CLK: now also U?.16 (SCLK)
- net SPI0_MISO: now also U?.15 (DOUT)
- net SPI0_MOSI: now also U?.14 (DIN)
- net SPI0_nCS: now also U?.1 (~CS)
- net at C49.1: now also U?.2 (VA)
- net at C50.1: now also U?.13 (VD)
Other:
- moved on the sheet: C48, C49, C50, R30, R31, R32, R35, U6
