File: asic/e-class-aardonyx/board/Board_Design/arduino_header.sch (KiCad schematic (older format))
At the start: 31 parts, among them J10 Conn_1x6_F, J11 Conn_1x6_F, J12 Conn_1x3_M, J13 Conn_1x8, J14 Conn_1x6_F, J15 Conn_1x10, J16 Conn_1x8, J7 Conn_1X4, J8 Conn_1x3_M, J9 Conn_1x8, U5 CAT24M01WI-GT3, U6 IS25LP256x-xM, U8 LSF0108PWR, U9 LSF0108PWR

Commit message: update bom
Parts:
- R36, R37: Description (none) -> RES 200K OHM 0.1% 1/16W 0402; Digikey PartNumber (none) -> 2019-RN73H1ETTP2003B25CT-ND; Manufactured Part Number (none) -> RN73H1ETTP2003B25; Maufaturer (none) -> KOA Speer Electronics, Inc.
- U5: Description (none) -> IC EEPROM 1M I2C 1MHZ 8SOIC; Digikey PartNumber (none) -> CAT24M01WI-GT3OSCT-ND; Manufactured Part Number (none) -> CAT24M01WI-GT3; Maufaturer (none) -> ON Semiconductor
- U6: Description (none) -> IC FLASH 256M SPI 133MHZ 16SOIC; Digikey PartNumber (none) -> 706-1611-ND; Manufactured Part Number (none) -> IS25LP256D-JMLE; Maufaturer (none) -> ISSI, Integrated Silicon Solution Inc
- U8, U9: Description (none) -> IC TRNSLTR BIDIRECTIONAL 20TSSOP; Digikey PartNumber (none) -> 296-37828-1-ND; Manufactured Part Number (none) -> LSF0108PWR; Maufaturer (none) -> Texas Instruments
- U?: Description (none) -> ADC108S102CIMTX/NOPB; Digikey PartNumber (none) -> 296-43835-1-ND; Manufactured Part Number (none) -> ADC108S102CIMTX/NOPB; Maufaturer (none) -> Texas Instruments
Changed lines of the file:
@@
 F 1 "IS25LP256x-xM" H 3150 1500 50  0000 C CNN
 F 2 "Package_SO:SOIC-16W_7.5x10.3mm_P1.27mm" H 2800 2550 50  0001 C CNN
-F 3 "" H 2800 1450 50  0001 C CNN
+F 3 "https://www.digikey.in/product-detail/en/issi-integrated-silicon-solution-inc/IS25LP256D-JMLE/706-1611-ND/7567432" H 2800 1450 50  0001 C CNN
+F 4 "IC FLASH 256M SPI 133MHZ 16SOIC" H 2750 1950 50  0001 C CNN "Description"
+F 5 "706-1611-ND" H 2750 1950 50  0001 C CNN "Digikey PartNumber"
+F 6 "IS25LP256D-JMLE" H 2750 1950 50  0001 C CNN "Manufactured Part Number"
+F 7 "ISSI, Integrated Silicon Solution Inc" H 2750 1950 50  0001 C CNN "Maufaturer"
 	1    2750 1950
 	1    0    0    -1
@@
 F 1 "CAT24M01WI-GT3" H 1900 5150 50  0000 C CNN
 F 2 "" H 1500 5650 50  0001 C CNN
-F 3 "" H 1500 5650 50  0001 C CNN
+F 3 "https://www.digikey.in/product-detail/en/on-semiconductor/CAT24M01WI-GT3/CAT24M01WI-GT3OSCT-ND/2698362" H 1500 5650 50  0001 C CNN
+F 4 "IC EEPROM 1M I2C 1MHZ 8SOIC" H 1500 5650 50  0001 C CNN "Description"
+F 5 "CAT24M01WI-GT3OSCT-ND" H 1500 5650 50  0001 C CNN "Digikey PartNumber"
+F 6 "CAT24M01WI-GT3" H 1500 5650 50  0001 C CNN "Manufactured Part Number"
+F 7 "ON Semiconductor" H 1500 5650 50  0001 C CNN "Maufaturer"
 	1    1500 5650
 	1    0    0    -1
@@
 F 1 "LSF0108PWR" H 10050 1850 50  0000 C CNN
 F 2 "" H 9750 2600 50  0001 C CNN
-F 3 "" H 9750 2600 50  0001 C CNN
+F 3 "https://www.digikey.in/product-detail/en/texas-instruments/LSF0108PWR/296-37828-1-ND/4876357" H 9750 2600 50  0001 C CNN
+F 4 "IC TRNSLTR BIDIRECTIONAL 20TSSOP" H 9750 2600 50  0001 C CNN "Description"
+F 5 "296-37828-1-ND" H 9750 2600 50  0001 C CNN "Digikey PartNumber"
+F 6 "LSF0108PWR" H 9750 2600 50  0001 C CNN "Manufactured Part Number"
+F 7 "Texas Instruments" H 9750 2600 50  0001 C CNN "Maufaturer"
 	1    9750 2600
 	1    0    0    -1
@@
 F 1 "200K" H 7018 1305 50  0000 L CNN
 F 2 "" V 6990 1340 50  0001 C CNN
-F 3 "~" H 6950 1350 50  0001 C CNN
+F 3 "https://www.digikey.com/product-detail/en/koa-speer-electronics-inc/RN73H1ETTP2003B25/2019-RN73H1ETTP2003B25CT-ND/9916930" H 6950 1350 50  0001 C CNN
+F 4 " RES 200K OHM 0.1% 1/16W 0402 " H 6950 1350 50  0001 C CNN "Description"
+F 5 "2019-RN73H1ETTP2003B25CT-ND " H 6950 1350 50  0001 C CNN "Digikey PartNumber"
+F 6 "RN73H1ETTP2003B25" H 6950 1350 50  0001 C CNN "Manufactured Part Number"
+F 7 "KOA Speer Electronics, Inc." H 6950 1350 50  0001 C CNN "Maufaturer"
 	1    6950 1350
 	1    0    0    -1
@@
 F 1 "200K" H 9968 1355 50  0000 L CNN
 F 2 "" V 9940 1390 50  0001 C CNN
-F 3 "~" H 9900 1400 50  0001 C CNN
+F 3 "https://www.digikey.com/product-detail/en/koa-speer-electronics-inc/RN73H1ETTP2003B25/2019-RN73H1ETTP2003B25CT-ND/9916930" H 9900 1400 50  0001 C CNN
+F 4 " RES 200K OHM 0.1% 1/16W 0402 " H 9900 1400 50  0001 C CNN "Description"
+F 5 "2019-RN73H1ETTP2003B25CT-ND " H 9900 1400 50  0001 C CNN "Digikey PartNumber"
+F 6 "RN73H1ETTP2003B25" H 9900 1400 50  0001 C CNN "Manufactured Part Number"
+F 7 "KOA Speer Electronics, Inc." H 9900 1400 50  0001 C CNN "Maufaturer"
 	1    9900 1400
 	1    0    0    -1
@@
 F 1 "LSF0108PWR" H 7100 1800 50  0000 C CNN
 F 2 "" H 6800 2550 50  0001 C CNN
-F 3 "" H 6800 2550 50  0001 C CNN
+F 3 "https://www.digikey.in/product-detail/en/texas-instruments/LSF0108PWR/296-37828-1-ND/4876357" H 6800 2550 50  0001 C CNN
+F 4 "IC TRNSLTR BIDIRECTIONAL 20TSSOP" H 6800 2550 50  0001 C CNN "Description"
+F 5 "296-37828-1-ND" H 6800 2550 50  0001 C CNN "Digikey PartNumber"
+F 6 "LSF0108PWR" H 6800 2550 50  0001 C CNN "Manufactured Part Number"
+F 7 "Texas Instruments" H 6800 2550 50  0001 C CNN "Maufaturer"
 	1    6800 2550
 	1    0    0    -1
@@
 F 1 "ADC108S102CIMTX" H 4750 5400 50  0000 C CNN
 F 2 "" H 4300 5900 50  0001 L BNN
-F 3 "" H 4300 5900 50  0001 L BNN
+F 3 "https://www.digikey.in/product-detail/en/texas-instruments/ADC108S102CIMTX-NOPB/296-43835-1-ND/5875706" H 4300 5900 50  0001 L BNN
+F 4 "ADC108S102CIMTX/NOPB" H 4300 5900 50  0001 C CNN "Description"
+F 5 "296-43835-1-ND" H 4300 5900 50  0001 C CNN "Digikey PartNumber"
+F 6 "ADC108S102CIMTX/NOPB" H 4300 5900 50  0001 C CNN "Manufactured Part Number"
+F 7 "Texas Instruments" H 4300 5900 50  0001 C CNN "Maufaturer"
 	1    4300 5900
 	1    0    0    -1

Commit message: update BOM
Parts:
- C47, C48, C49, C50, C51, C52, C53, C54: Description CAP CER 0.1UF 16V X7R 0402 -> CAP CER 0.1UF 25V X7R 0402; Digikey PartNumber 490-6328-1-ND -> 478-10050-1-ND; Manufactured Part Number GRM155R71C104KA88J -> 04023C104JAT2A; Maufaturer Murata -> AVX Corporation
Changed lines of the file:
@@
 F 1 "0.1UF" H 7642 1255 50  0000 L CNN
 F 2 "" H 7550 1300 50  0001 C CNN
-F 3 "https://www.digikey.in/product-detail/en/murata-electronics/GRM155R71C104KA88J/490-6328-1-ND/3845525" H 7550 1300 50  0001 C CNN
-F 4 "CAP CER 0.1UF 16V X7R 0402 " H 7550 1300 50  0001 C CNN "Description"
-F 5 " 490-6328-1-ND " H 7550 1300 50  0001 C CNN "Digikey PartNumber"
-F 6 "GRM155R71C104KA88J " H 7550 1300 50  0001 C CNN "Manufactured Part Number"
-F 7 "Murata" H 7550 1300 50  0001 C CNN "Maufaturer"
+F 3 "https://www.digikey.in/product-detail/en/avx-corporation/04023C104JAT2A/478-10050-1-ND/6564273" H 7550 1300 50  0001 C CNN
+F 4 "CAP CER 0.1UF 25V X7R 0402" H 7550 1300 50  0001 C CNN "Description"
+F 5 "478-10050-1-ND" H 7550 1300 50  0001 C CNN "Digikey PartNumber"
+F 6 "04023C104JAT2A" H 7550 1300 50  0001 C CNN "Manufactured Part Number"
+F 7 "AVX Corporation" H 7550 1300 50  0001 C CNN "Maufaturer"
 	1    7550 1300
 	1    0    0    -1
@@
 F 1 "0.1UF" H 9242 1305 50  0000 L CNN
 F 2 "" H 9150 1350 50  0001 C CNN
-F 3 "https://www.digikey.in/product-detail/en/murata-electronics/GRM155R71C104KA88J/490-6328-1-ND/3845525" H 9150 1350 50  0001 C CNN
-F 4 "CAP CER 0.1UF 16V X7R 0402 " H 9150 1350 50  0001 C CNN "Description"
-F 5 " 490-6328-1-ND " H 9150 1350 50  0001 C CNN "Digikey PartNumber"
-F 6 "GRM155R71C104KA88J " H 9150 1350 50  0001 C CNN "Manufactured Part Number"
-F 7 "Murata" H 9150 1350 50  0001 C CNN "Maufaturer"
+F 3 "https://www.digikey.in/product-detail/en/avx-corporation/04023C104JAT2A/478-10050-1-ND/6564273" H 9150 1350 50  0001 C CNN
+F 4 "CAP CER 0.1UF 25V X7R 0402" H 9150 1350 50  0001 C CNN "Description"
+F 5 "478-10050-1-ND" H 9150 1350 50  0001 C CNN "Digikey PartNumber"
+F 6 "04023C104JAT2A" H 9150 1350 50  0001 C CNN "Manufactured Part Number"
+F 7 "AVX Corporation" H 9150 1350 50  0001 C CNN "Maufaturer"
 	1    9150 1350
 	1    0    0    -1
@@
 F 1 "0.1UF" H 6342 1255 50  0000 L CNN
 F 2 "" H 6250 1300 50  0001 C CNN
-F 3 "https://www.digikey.in/product-detail/en/murata-electronics/GRM155R71C104KA88J/490-6328-1-ND/3845525" H 6250 1300 50  0001 C CNN
-F 4 "CAP CER 0.1UF 16V X7R 0402 " H 6250 1300 50  0001 C CNN "Description"
-F 5 " 490-6328-1-ND " H 6250 1300 50  0001 C CNN "Digikey PartNumber"
-F 6 "GRM155R71C104KA88J " H 6250 1300 50  0001 C CNN "Manufactured Part Number"
-F 7 "Murata" H 6250 1300 50  0001 C CNN "Maufaturer"
+F 3 "https://www.digikey.in/product-detail/en/avx-corporation/04023C104JAT2A/478-10050-1-ND/6564273" H 6250 1300 50  0001 C CNN
+F 4 "CAP CER 0.1UF 25V X7R 0402" H 6250 1300 50  0001 C CNN "Description"
+F 5 "478-10050-1-ND" H 6250 1300 50  0001 C CNN "Digikey PartNumber"
+F 6 "04023C104JAT2A" H 6250 1300 50  0001 C CNN "Manufactured Part Number"
+F 7 "AVX Corporation" H 6250 1300 50  0001 C CNN "Maufaturer"
 	1    6250 1300
 	1    0    0    -1
@@
 F 1 "0.1UF " H 10592 1305 50  0000 L CNN
 F 2 "" H 10500 1350 50  0001 C CNN
-F 3 "https://www.digikey.in/product-detail/en/murata-electronics/GRM155R71C104KA88J/490-6328-1-ND/3845525" H 10500 1350 50  0001 C CNN
-F 4 "CAP CER 0.1UF 16V X7R 0402 " H 10500 1350 50  0001 C CNN "Description"
-F 5 " 490-6328-1-ND " H 10500 1350 50  0001 C CNN "Digikey PartNumber"
-F 6 "GRM155R71C104KA88J " H 10500 1350 50  0001 C CNN "Manufactured Part Number"
-F 7 "Murata" H 10500 1350 50  0001 C CNN "Maufaturer"
+F 3 "https://www.digikey.in/product-detail/en/avx-corporation/04023C104JAT2A/478-10050-1-ND/6564273" H 10500 1350 50  0001 C CNN
+F 4 "CAP CER 0.1UF 25V X7R 0402" H 10500 1350 50  0001 C CNN "Description"
+F 5 "478-10050-1-ND" H 10500 1350 50  0001 C CNN "Digikey PartNumber"
+F 6 "04023C104JAT2A" H 10500 1350 50  0001 C CNN "Manufactured Part Number"
+F 7 "AVX Corporation" H 10500 1350 50  0001 C CNN "Maufaturer"
 	1    10500 1350
 	1    0    0    -1
@@
 F 1 "0.1UF" H 3392 1155 50  0000 L CNN
 F 2 "" H 3300 1200 50  0001 C CNN
-F 3 "https://www.digikey.in/product-detail/en/murata-electronics/GRM155R71C104KA88J/490-6328-1-ND/3845525" H 3300 1200 50  0001 C CNN
-F 4 "CAP CER 0.1UF 16V X7R 0402 " H 3300 1200 50  0001 C CNN "Description"
-F 5 " 490-6328-1-ND " H 3300 1200 50  0001 C CNN "Digikey PartNumber"
-F 6 "GRM155R71C104KA88J " H 3300 1200 50  0001 C CNN "Manufactured Part Number"
-F 7 "Murata" H 3300 1200 50  0001 C CNN "Maufaturer"
+F 3 "https://www.digikey.in/product-detail/en/avx-corporation/04023C104JAT2A/478-10050-1-ND/6564273" H 3300 1200 50  0001 C CNN
+F 4 "CAP CER 0.1UF 25V X7R 0402" H 3300 1200 50  0001 C CNN "Description"
+F 5 "478-10050-1-ND" H 3300 1200 50  0001 C CNN "Digikey PartNumber"
+F 6 "04023C104JAT2A" H 3300 1200 50  0001 C CNN "Manufactured Part Number"
+F 7 "AVX Corporation" H 3300 1200 50  0001 C CNN "Maufaturer"
 	1    3300 1200
 	1    0    0    -1
@@
 F 1 "0.1UF" H 2142 4955 50  0000 L CNN
 F 2 "" H 2050 5000 50  0001 C CNN
-F 3 "https://www.digikey.in/product-detail/en/murata-electronics/GRM155R71C104KA88J/490-6328-1-ND/3845525" H 2050 5000 50  0001 C CNN
-F 4 "CAP CER 0.1UF 16V X7R 0402 " H 2050 5000 50  0001 C CNN "Description"
-F 5 " 490-6328-1-ND " H 2050 5000 50  0001 C CNN "Digikey PartNumber"
-F 6 "GRM155R71C104KA88J " H 2050 5000 50  0001 C CNN "Manufactured Part Number"
-F 7 "Murata" H 2050 5000 50  0001 C CNN "Maufaturer"
+F 3 "https://www.digikey.in/product-detail/en/avx-corporation/04023C104JAT2A/478-10050-1-ND/6564273" H 2050 5000 50  0001 C CNN
+F 4 "CAP CER 0.1UF 25V X7R 0402" H 2050 5000 50  0001 C CNN "Description"
+F 5 "478-10050-1-ND" H 2050 5000 50  0001 C CNN "Digikey PartNumber"
+F 6 "04023C104JAT2A" H 2050 5000 50  0001 C CNN "Manufactured Part Number"
+F 7 "AVX Corporation" H 2050 5000 50  0001 C CNN "Maufaturer"
 	1    2050 5000
 	1    0    0    -1
@@
 F 1 "0.1UF" H 4992 5005 50  0000 L CNN
 F 2 "" H 4900 5050 50  0001 C CNN
-F 3 "https://www.digikey.in/product-detail/en/murata-electronics/GRM155R71C104KA88J/490-6328-1-ND/3845525" H 4900 5050 50  0001 C CNN
-F 4 "CAP CER 0.1UF 16V X7R 0402 " H 4900 5050 50  0001 C CNN "Description"
-F 5 " 490-6328-1-ND " H 4900 5050 50  0001 C CNN "Digikey PartNumber"
-F 6 "GRM155R71C104KA88J " H 4900 5050 50  0001 C CNN "Manufactured Part Number"
-F 7 "Murata" H 4900 5050 50  0001 C CNN "Maufaturer"
+F 3 "https://www.digikey.in/product-detail/en/avx-corporation/04023C104JAT2A/478-10050-1-ND/6564273" H 4900 5050 50  0001 C CNN
+F 4 "CAP CER 0.1UF 25V X7R 0402" H 4900 5050 50  0001 C CNN "Description"
+F 5 "478-10050-1-ND" H 4900 5050 50  0001 C CNN "Digikey PartNumber"
+F 6 "04023C104JAT2A" H 4900 5050 50  0001 C CNN "Manufactured Part Number"
+F 7 "AVX Corporation" H 4900 5050 50  0001 C CNN "Maufaturer"
 	1    4900 5050
 	1    0    0    -1
@@
 F 1 "0.1UF" H 3792 5005 50  0000 L CNN
 F 2 "" H 3700 5050 50  0001 C CNN
-F 3 "https://www.digikey.in/product-detail/en/murata-electronics/GRM155R71C104KA88J/490-6328-1-ND/3845525" H 3700 5050 50  0001 C CNN
-F 4 "CAP CER 0.1UF 16V X7R 0402 " H 3700 5050 50  0001 C CNN "Description"
-F 5 " 490-6328-1-ND " H 3700 5050 50  0001 C CNN "Digikey PartNumber"
-F 6 "GRM155R71C104KA88J " H 3700 5050 50  0001 C CNN "Manufactured Part Number"
-F 7 "Murata" H 3700 5050 50  0001 C CNN "Maufaturer"
+F 3 "https://www.digikey.in/product-detail/en/avx-corporation/04023C104JAT2A/478-10050-1-ND/6564273" H 3700 5050 50  0001 C CNN
+F 4 "CAP CER 0.1UF 25V X7R 0402" H 3700 5050 50  0001 C CNN "Description"
+F 5 "478-10050-1-ND" H 3700 5050 50  0001 C CNN "Digikey PartNumber"
+F 6 "04023C104JAT2A" H 3700 5050 50  0001 C CNN "Manufactured Part Number"
+F 7 "AVX Corporation" H 3700 5050 50  0001 C CNN "Maufaturer"
 	1    3700 5050
 	-1   0    0    -1

Commit message: updated BOM
Parts:
- C47, C48, C49, C50, C51, C52, C53, C54: value 0.1UF -> 0.1UF,0402
- J10, J11, J14: Description (none) -> CONN RCPT 6POS 0.1 GOLD PCB; Digikey PartNumber (none) -> 609-3558-ND; Manufactured Part Number (none) -> 75915-306LF; Maufaturer (none) -> Amphenol ICC (FCI)
- J12, J8: Description (none) -> CONN HEADER VERT 3POS 2.54MM; Digikey PartNumber (none) -> 609-3464-ND; Manufactured Part Number (none) -> 68000-203HLF; Maufaturer (none) -> Amphenol ICC (FCI)
- J13: value Conn_1x8 -> Conn_1x8_F; Description (none) -> CONN RCPT 8POS 0.1 GOLD PCB; Digikey PartNumber (none) -> 609-3264-ND; Field4 (none) -> 609-3589-ND; Manufactured Part Number (none) -> 68685-308LF; Maufaturer (none) -> Amphenol ICC (FCI)
- J15: Description (none) -> CONN RCPT 10POS 0.1 GOLD PCB; Digikey PartNumber (none) -> 609-3584-ND; Manufactured Part Number (none) -> 68685-310LF; Maufaturer (none) -> Amphenol ICC (FCI)
- J16: value Conn_1x8 -> Conn_1x8_F; Description (none) -> CONN RCPT 8POS 0.1 GOLD PCB; Digikey PartNumber (none) -> 609-3264-ND; Manufactured Part Number (none) -> 68685-308LF; Maufaturer (none) -> Amphenol ICC (FCI)
- J7: value Conn_1X4 -> Conn_1x4; Description (none) -> CONN HEADER VERT 4POS 2.54MM; Digikey PartNumber (none) -> 609-3262-ND; Manufactured Part Number (none) -> 68000-404HLF; Maufaturer (none) -> Amphenol ICC (FCI)
- J9: Description (none) -> CONN HEADER VERT 8POS 2.54MM; Digikey PartNumber (none) -> 609-3264-ND; Manufactured Part Number (none) -> 68000-408HLF; Maufaturer (none) -> Amphenol ICC (FCI)
- R30, R31, R32, R33, R34, R35: value 10K -> 10KE,0805
- R36, R37: value 200K -> 200KE,0402
- gave numbers to parts that had none: 1
