File: asic/e-class-aardonyx/board/Board_Design/power_2.sch (KiCad schematic (older format))
At the start: 36 parts, among them Q1 FDN339AN, SW2 FSM2JSMAATR, U10 TPS7A7002DDAR, U11 ADM1085, U12 ADM1085, U13 TPS7A7002DDAR, U14 74AUP1G09GW

Commit message: update bom
Parts:
- D4, D5: Description (none) -> LED GREEN DIFFUSED 1206 SMD; Digikey PartNumber (none) -> 67-1002-1-ND; Manufactured Part Number (none) -> SML-LX1206GW-TR; Maufaturer (none) -> Lumex Opto/Components Inc.
- Q1: Description (none) -> MOSFET N-CH 20V 3A SSOT3; Digikey PartNumber (none) -> FDN339ANCT-ND; Manufactured Part Number (none) -> FDN339AN; Maufaturer (none) -> ON Semiconductor
- R39, R40, R47, R54: Description (none) -> RES SMD 0 OHM JUMPER 1/8W 0805; Digikey PartNumber (none) -> 541-0.0ACT-ND; Manufactured Part Number (none) -> CRCW08050000Z0EA; Maufaturer (none) -> Vishay Dale
- R41: Description (none) -> RES 169K OHM 0.1% 1/8W 0805; Digikey PartNumber (none) -> P169KDACT-ND; Manufactured Part Number (none) -> ERA-6AEB1693V; Maufaturer (none) -> Panasonic Electronic Components
- U10, U13: Description (none) -> IC REG LIN POS ADJ 3A 8SO PWRPAD; Digikey PartNumber (none) -> 296-40977-1-ND; Manufactured Part Number (none) -> TPS7A7002DDAR; Maufaturer (none) -> Texas Instruments
- U11, U12: Description (none) -> IC SUPERVISOR 1 CHANNEL SC70-6; Digikey PartNumber (none) -> ADM1085AKSZ-REEL7CT-ND; Manufactured Part Number (none) -> ADM1085AKSZ-REEL7; Maufaturer (none) -> Analog Devices Inc.
- U14: Description (none) -> IC GATE AND 1CH 2-INP 5TSSOP; Digikey PartNumber (none) -> 1727-4492-1-ND; Manufactured Part Number (none) -> 74AUP1G09GW,125; Maufaturer (none) -> Nexperia USA Inc.
Changed lines of the file:
@@
 F 1 "169K" H 3068 1805 50  0000 L CNN
 F 2 "" V 3040 1840 50  0001 C CNN
-F 3 "~" H 3000 1850 50  0001 C CNN
+F 3 "https://www.digikey.com/product-detail/en/panasonic-electronic-components/ERA-6AEB1693V/P169KDACT-ND/3074985" H 3000 1850 50  0001 C CNN
+F 4 "RES 169K OHM 0.1% 1/8W 0805" H 3000 1850 50  0001 C CNN "Description"
+F 5 "P169KDACT-ND" H 3000 1850 50  0001 C CNN "Digikey PartNumber"
+F 6 "ERA-6AEB1693V" H 3000 1850 50  0001 C CNN "Manufactured Part Number"
+F 7 "Panasonic Electronic Components" H 3000 1850 50  0001 C CNN "Maufaturer"
 	1    3000 1850
 	1    0    0    -1
@@
 F 1 "SML-LX1206GW" V 4150 2050 50  0000 R CNN
 F 2 "" H 4400 2100 50  0001 C CNN
-F 3 "~" H 4400 2100 50  0001 C CNN
+F 3 "https://www.digikey.in/product-detail/en/lumex-opto-components-inc/SML-LX1206GW-TR/67-1002-1-ND/270799" H 4400 2100 50  0001 C CNN
+F 4 "LED GREEN DIFFUSED 1206 SMD" H 4400 2100 50  0001 C CNN "Description"
+F 5 "67-1002-1-ND" H 4400 2100 50  0001 C CNN "Digikey PartNumber"
+F 6 "SML-LX1206GW-TR" H 4400 2100 50  0001 C CNN "Manufactured Part Number"
+F 7 "Lumex Opto/Components Inc." H 4400 2100 50  0001 C CNN "Maufaturer"
 	1    4400 2100
 	0    -1   -1   0
@@
 F 1 "ADM1085" H 3450 4350 50  0000 C CNN
 F 2 "" H 3100 4750 50  0001 C CNN
-F 3 "" H 3100 4750 50  0001 C CNN
+F 3 "https://www.digikey.in/product-detail/en/analog-devices-inc/ADM1085AKSZ-REEL7/ADM1085AKSZ-REEL7CT-ND/820429" H 3100 4750 50  0001 C CNN
+F 4 "IC SUPERVISOR 1 CHANNEL SC70-6" H 3200 4700 50  0001 C CNN "Description"
+F 5 "ADM1085AKSZ-REEL7CT-ND" H 3200 4700 50  0001 C CNN "Digikey PartNumber"
+F 6 "ADM1085AKSZ-REEL7" H 3200 4700 50  0001 C CNN "Manufactured Part Number"
+F 7 "Analog Devices Inc." H 3200 4700 50  0001 C CNN "Maufaturer"
 	1    3200 4700
 	1    0    0    -1
@@
 F 1 "TPS7A7002DDAR" H 2300 2474 50  0000 C CNN
 F 2 "" H 2300 1950 50  0001 C CNN
-F 3 "" H 2300 1950 50  0001 C CNN
+F 3 "https://www.digikey.in/product-detail/en/texas-instruments/TPS7A7002DDAR/296-40977-1-ND/5178854" H 2300 1950 50  0001 C CNN
+F 4 "IC REG LIN POS ADJ 3A 8SO PWRPAD" H 2300 1950 50  0001 C CNN "Description"
+F 5 "296-40977-1-ND" H 2300 1950 50  0001 C CNN "Digikey PartNumber"
+F 6 "TPS7A7002DDAR" H 2300 1950 50  0001 C CNN "Manufactured Part Number"
+F 7 "Texas Instruments" H 2300 1950 50  0001 C CNN "Maufaturer"
 	1    2300 1950
 	1    0    0    -1
@@
 F 1 "TPS7A7002DDAR" H 7950 2674 50  0000 C CNN
 F 2 "" H 7950 2150 50  0001 C CNN
-F 3 "" H 7950 2150 50  0001 C CNN
+F 3 "https://www.digikey.in/product-detail/en/texas-instruments/TPS7A7002DDAR/296-40977-1-ND/5178854" H 7950 2150 50  0001 C CNN
+F 4 "IC REG LIN POS ADJ 3A 8SO PWRPAD" H 7950 2150 50  0001 C CNN "Description"
+F 5 "296-40977-1-ND" H 7950 2150 50  0001 C CNN "Digikey PartNumber"
+F 6 "TPS7A7002DDAR" H 7950 2150 50  0001 C CNN "Manufactured Part Number"
+F 7 "Texas Instruments" H 7950 2150 50  0001 C CNN "Maufaturer"
 	1    7950 2150
 	1    0    0    -1
@@
 F 1 "SML-LX1206GW" V 10250 1900 50  0000 R CNN
 F 2 "" H 10350 2050 50  0001 C CNN
-F 3 "~" H 10350 2050 50  0001 C CNN
+F 3 "https://www.digikey.in/product-detail/en/lumex-opto-components-inc/SML-LX1206GW-TR/67-1002-1-ND/270799" H 10350 2050 50  0001 C CNN
+F 4 "LED GREEN DIFFUSED 1206 SMD" H 10350 2050 50  0001 C CNN "Description"
+F 5 "67-1002-1-ND" H 10350 2050 50  0001 C CNN "Digikey PartNumber"
+F 6 "SML-LX1206GW-TR" H 10350 2050 50  0001 C CNN "Manufactured Part Number"
+F 7 "Lumex Opto/Components Inc." H 10350 2050 50  0001 C CNN "Maufaturer"
 	1    10350 2050
 	0    -1   -1   0
@@
 F 1 "0E" V 2450 4800 50  0000 L CNN
 F 2 "" V 2590 4790 50  0001 C CNN
-F 3 "~" H 2550 4800 50  0001 C CNN
+F 3 "https://www.digikey.com/product-detail/en/vishay-dale/CRCW08050000Z0EA/541-0-0ACT-ND/1180267" H 2550 4800 50  0001 C CNN
+F 4 " RES SMD 0 OHM JUMPER 1/8W 0805 " H 2550 4800 50  0001 C CNN "Description"
+F 5 " 541-0.0ACT-ND " H 2550 4800 50  0001 C CNN "Digikey PartNumber"
+F 6 " CRCW08050000Z0EA " H 2550 4800 50  0001 C CNN "Manufactured Part Number"
+F 7 "Vishay Dale" H 2550 4800 50  0001 C CNN "Maufaturer"
 	1    2550 4800
 	0    -1   -1   0
@@
 F 1 "FDN339AN" H 10448 2455 50  0000 L CNN
 F 2 "SSOT-3" H 10350 2500 50  0001 L BNN
-F 3 "" H 10350 2500 50  0001 C CNN
+F 3 "https://www.digikey.in/product-detail/en/on-semiconductor/FDN339AN/FDN339ANCT-ND/965603" H 10350 2500 50  0001 C CNN
+F 4 "MOSFET N-CH 20V 3A SSOT3" H 10350 2500 50  0001 C CNN "Description"
+F 5 "FDN339ANCT-ND" H 10350 2500 50  0001 C CNN "Digikey PartNumber"
+F 6 "FDN339AN" H 10350 2500 50  0001 C CNN "Manufactured Part Number"
+F 7 "ON Semiconductor" H 10350 2500 50  0001 C CNN "Maufaturer"
 	1    10350 2500
 	1    0    0    -1
@@
 F 1 "ADM1085" H 3500 6150 50  0000 C CNN
 F 2 "" H 3150 6550 50  0001 C CNN
-F 3 "" H 3150 6550 50  0001 C CNN
+F 3 "https://www.digikey.in/product-detail/en/analog-devices-inc/ADM1085AKSZ-REEL7/ADM1085AKSZ-REEL7CT-ND/820429" H 3150 6550 50  0001 C CNN
+F 4 "IC SUPERVISOR 1 CHANNEL SC70-6" H 3250 6500 50  0001 C CNN "Description"
+F 5 "ADM1085AKSZ-REEL7CT-ND" H 3250 6500 50  0001 C CNN "Digikey PartNumber"
+F 6 "ADM1085AKSZ-REEL7" H 3250 6500 50  0001 C CNN "Manufactured Part Number"
+F 7 "Analog Devices Inc." H 3250 6500 50  0001 C CNN "Maufaturer"
 	1    3250 6500
 	1    0    0    -1
@@
 F 1 "0E" V 2500 6600 50  0000 L CNN
 F 2 "" V 2640 6590 50  0001 C CNN
-F 3 "~" H 2600 6600 50  0001 C CNN
+F 3 "https://www.digikey.com/product-detail/en/vishay-dale/CRCW08050000Z0EA/541-0-0ACT-ND/1180267" H 2600 6600 50  0001 C CNN
+F 4 " RES SMD 0 OHM JUMPER 1/8W 0805 " H 2600 6600 50  0001 C CNN "Description"
+F 5 " 541-0.0ACT-ND " H 2600 6600 50  0001 C CNN "Digikey PartNumber"
+F 6 " CRCW08050000Z0EA " H 2600 6600 50  0001 C CNN "Manufactured Part Number"
+F 7 "Vishay Dale" H 2600 6600 50  0001 C CNN "Maufaturer"
 	1    2600 6600
 	0    -1   -1   0
@@
 F 1 "74AUP1G09GW" H 9550 5150 50  0000 C CNN
 F 2 "" H 9250 5300 50  0001 C CNN
-F 3 "" H 9250 5300 50  0001 C CNN
+F 3 "https://www.digikey.in/product-detail/en/nexperia-usa-inc/74AUP1G09GW-125/1727-4492-1-ND/2530869" H 9250 5300 50  0001 C CNN
+F 4 "IC GATE AND 1CH 2-INP 5TSSOP" H 9250 5300 50  0001 C CNN "Description"
+F 5 "1727-4492-1-ND" H 9250 5300 50  0001 C CNN "Digikey PartNumber"
+F 6 "74AUP1G09GW,125" H 9250 5300 50  0001 C CNN "Manufactured Part Number"
+F 7 "Nexperia USA Inc." H 9250 5300 50  0001 C CNN "Maufaturer"
 	1    9250 5300
 	1    0    0    -1
@@
 F 1 "0E" V 9950 5300 50  0000 L CNN
 F 2 "" V 10090 5290 50  0001 C CNN
-F 3 "~" H 10050 5300 50  0001 C CNN
+F 3 "https://www.digikey.com/product-detail/en/vishay-dale/CRCW08050000Z0EA/541-0-0ACT-ND/1180267" H 10050 5300 50  0001 C CNN
+F 4 " RES SMD 0 OHM JUMPER 1/8W 0805 " H 10050 5300 50  0001 C CNN "Description"
+F 5 " 541-0.0ACT-ND " H 10050 5300 50  0001 C CNN "Digikey PartNumber"
+F 6 " CRCW08050000Z0EA " H 10050 5300 50  0001 C CNN "Manufactured Part Number"
+F 7 "Vishay Dale" H 10050 5300 50  0001 C CNN "Maufaturer"
 	1    10050 5300
 	0    -1   -1   0
@@
 F 1 "0E" V 8200 6200 50  0000 L CNN
 F 2 "" V 8340 6190 50  0001 C CNN
-F 3 "~" H 8300 6200 50  0001 C CNN
+F 3 "https://www.digikey.com/product-detail/en/vishay-dale/CRCW08050000Z0EA/541-0-0ACT-ND/1180267" H 8300 6200 50  0001 C CNN
+F 4 " RES SMD 0 OHM JUMPER 1/8W 0805 " H 8300 6200 50  0001 C CNN "Description"
+F 5 " 541-0.0ACT-ND " H 8300 6200 50  0001 C CNN "Digikey PartNumber"
+F 6 " CRCW08050000Z0EA " H 8300 6200 50  0001 C CNN "Manufactured Part Number"
+F 7 "Vishay Dale" H 8300 6200 50  0001 C CNN "Maufaturer"
 	1    8300 6200
 	0    -1   -1   0

Commit message: update BOM
Parts:
- C56, C62: Description CAP CER 10UF 16V X5R 0805 -> CAP CER 10UF 25V X7R 1206; Digikey PartNumber 490-6473-1-ND -> 399-15734-1-ND; Manufactured Part Number GRM21BR61C106KE15K -> C1206C106J3RACAUTO; Maufaturer Murata -> KEMET
- C57, C58: Description CAP CER 15PF 16V C0G/NP0 0402 -> CAP CER 15PF 25V C0G/NP0 0805; Digikey PartNumber 399-8947-1-ND -> 732-7828-1-ND; Manufactured Part Number C0402C150J4GACTU -> 885012007029; Maufaturer Kemet -> Würth Elektronik
- C60, C61: Description CAP CER 0.1UF 16V X7R 0402 -> CAP CER 0.1UF 25V X7R 0402; Digikey PartNumber 490-6328-1-ND -> 478-10050-1-ND; Manufactured Part Number GRM155R71C104KA88J -> 04023C104JAT2A; Maufaturer Murata -> AVX Corporation
- P_R52: renamed from R52; Description RES SMD 1K OHM 5% 1/10W 0402 -> RES SMD 1K OHM 5% 1/8W 0805; Digikey PartNumber P1.0KJCT-ND -> 311-1.0KARCT-ND; Manufactured Part Number ERA-2AEB123X -> RC0805JR-071KL; Maufaturer Panasonic Electronic Components -> Yageo
- P_R53: renamed from R53; Description RES SMD 1K OHM 5% 1/10W 0402 -> RES SMD 1K OHM 5% 1/8W 0805; Digikey PartNumber P1.0KJCT-ND -> 311-1.0KARCT-ND; Manufactured Part Number ERA-2AEB123X -> RC0805JR-071KL; Maufaturer Panasonic Electronic Components -> Yageo
- R47, R54: Description RES SMD 0 OHM JUMPER 1/8W 0805 -> RES SMD 0 OHM JUMPER 1/16W 0402; Digikey PartNumber 541-0.0ACT-ND -> 541-0.0JCT-ND; Manufactured Part Number CRCW08050000Z0EA -> CRCW04020000Z0ED
- renumbered R38 to P_R38, R39 to P_R39, R40 to P_R40, R41 to P_R41, R42 to P_R42, R43 to P_R43, R44 to P_R44, R49 to P_R49, R50 to P_R50, R56 to P_R56

Commit message: updated BOM
Parts:
- C55, C59: value 4.7UF -> 4.7UF,1206
- C56, C62: value 10UF -> 10UF,1206
- C57, C58: value 15pf -> 15PF,0805; Maufaturer Würth Elektronik -> Wurth Elektronik
- C60, C61: value 0.1UF -> 0.1UF,0402
- D4, D5: value SML-LX1206GW -> LED,0603; Description LED GREEN DIFFUSED 1206 SMD -> LED GREEN CLEAR CHIP SMD; Digikey PartNumber 67-1002-1-ND -> 160-1832-1-ND; Manufactured Part Number SML-LX1206GW-TR -> LTST-C193TGKT-5A; Maufaturer Lumex Opto/Components Inc. -> Lite-On Inc.
- P_R38, P_R43, R48, R51, R55: value 10K -> 10KE,0805
- P_R39, P_R40: value 0E -> 0E, 0805
- P_R41: value 169K -> 169KE,0805
- P_R42, P_R50: value 30.1K -> 30.1KE,0805
- P_R49: value 78.7K -> 78.7KE,0805
- P_R52, P_R53: value 1K -> 1KE,0805
- R45: value 4.7K -> 4.7KE, 0402
- R46: value 1K -> 1KE,0402
- R47, R54: value 0E -> 0E, 0402
- SW2: Description (none) -> SWITCH TACTILE SPST-NO 0.05A 24V; Digikey PartNumber (none) -> 450-1792-1-ND; Manufactured Part Number (none) -> FSM2JSMAATR; Maufaturer (none) -> TE Connectivity ALCOSWITCH Switches
