File: asic/e-class-aardonyx/board/Board_Design/Aardonyx_V01.kicad_pcb (KiCad board)
At the start: 4 copper layers, 298 parts, among them J1 USB_B_6PIN, J10 Conn_1x6_F, J11 Conn_1x6_F, J12 Conn_1x3_M, J13 Conn_1x8_F, J14 Conn_1x6_F, J15 Conn_1x10, J16 Conn_1x8_F, J17 USB_OTG, J18 Conn_1x3_M, J19 Conn_1x3_M, J2 Conn_1x8, J3 Conn_1x3_M, J4 Conn_1x4, J5 PJ-202H PWRJACK, J6 Conn_1x3_M, J7 Conn_1x4, J8 Conn_1x3_M, J9 Conn_1x8, Q1 FDN339AN, SW1 SW_SPST, SW2 FSM2JSMAATR, SW3 SW_DIP_x03, U1 FT2232H, U10 TPS7A7002DDAR, U11 ADM1085, U12 ADM1085, U13 TPS7A7002DDAR, U14 74AUP1G09GW, U15 SKT32E, U16 93LC56BT-I_OT, U2 IS42S32160F-TSOP2, U3 CDCE913PW, U4 TPS54627DDAR, U5 CAT24M01WI-GT3, U6 IS25LP256x-xM, U7 ADC108S102CIMTX, U8 LSF0108PWR, U9 LSF0108PWR, Y1 12MHz, Y2 27MHz

Commit message: updated components
Parts:
- C18, C19, C20, C21, C26, C28, C29, C64, C65, C66, C67, C68, C69, C70, C71, C72, C73, C74, C75, C76, C77, C78, C79, C80, C81, C82, C83, C84, C86, C87, C88, C89, C90, R20: moved to B.Cu
- C48, R100, R101, R102, R103, R104, R105, R106, R107, R108, R109, R110, R111, R112, R113, R114, R115, R116, R117, R118, R119, R120, R121, R122, R123, R124, R125, R126, R127, R65, R66, R67, R68, R69, R70, R71, R72, R73, R74, R75, R76, R77, R78, R79, R80, R81, R82, R83, R84, R85, R86, R87, R88, R89, R90, R91, R92, R93, R94, R95, R96, R97, R98, R99, U15, U2: moved to F.Cu
- moved R88 56.7 mm to (142.5, 147.6), turned to 270 degrees
- moved R83 56.7 mm to (139.0, 147.6), turned to 270 degrees
- moved R82 56.7 mm to (140.1, 147.6), turned to 270 degrees
- moved R89 56.7 mm to (141.3, 147.6), turned to 270 degrees
- moved R78 56.6 mm to (137.9, 147.6), turned to 270 degrees
- moved R79 56.6 mm to (136.7, 147.6), turned to 270 degrees
- moved C26 56.5 mm to (128.1, 91.0)
- moved C20 56.5 mm to (139.6, 91.0)
- moved R80 56.4 mm to (135.7, 147.5), turned to 270 degrees
- moved R81 56.1 mm to (132.2, 147.3), turned to 270 degrees
- moved R87 56.1 mm to (131.1, 147.3), turned to 270 degrees
- moved R86 56.0 mm to (129.9, 147.3), turned to 270 degrees
- moved R85 56.0 mm to (128.8, 147.3), turned to 270 degrees
- moved C21 56.0 mm to (133.7, 91.2)
- moved C29 56.0 mm to (131.1, 91.2), turned to 270 degrees
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